File: DC_motor_board/Pump_Control.kicad_sch (KiCad schematic)
At the start: 1 part, among them U4 ULN2003D1013TR

Commit message: Modify Pump Schems and PCB1
Parts:
- U4: value ULN2003D1013TR -> ULN2003D1013TR (SO-16)
Connections:
- net GNDD: now reaches U4.8 (GND)
Changed lines of the file:
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@@
     (effects (font (size 1.27 1.27)) (justify right))
+  )
+  (symbol (lib_id "power:GNDD") (at 120.65 102.87 0) (unit 1)
+    (in_bom yes) (on_board yes) (dnp no)
+    (property "Reference" "#PWR024" (at 120.65 109.22 0)
+      (effects (font (size 1.27 1.27)) hide)
+    )
+    (property "Value" "GNDD" (at 120.65 106.68 0)
+      (effects (font (size 1.27 1.27)))
+    )
+    (property "Footprint" "" (at 120.65 102.87 0)
+      (effects (font (size 1.27 1.27)) hide)
+    )
+    (property "Datasheet" "" (at 120.65 102.87 0)
+      (effects (font (size 1.27 1.27)) hide)
+    )
+    (pin "1")
+    (instances
+      (project "Плата насосов"
+        (path "/7f8f7dc9-8c50-44ed-985c-35a6d8c67be0"
+          (reference "#PWR024") (unit 1)
+        )
+        (path "/7f8f7dc9-8c50-44ed-985c-35a6d8c67be0/1b51a03a-fa78-498a-9890-137b4373474b"
+          (reference "#PWR052") (unit 1)
+        )
+      )
+    )
   )
   (symbol (lib_id "Transistor_Array:ULN2003") (at 120.65 87.63 0) (mirror y) (unit 1)
@@
       (effects (font (size 1.27 1.27)))
     )
-    (property "Value" "ULN2003D1013TR" (at 120.65 72.39 0)
+    (property "Value" "ULN2003D1013TR (SO-16)" (at 120.65 72.39 0)
       (effects (font (size 1.27 1.27)))
     )

Commit message: Modify Mian controller, stepmotor, motor 25.05.24
Connections:
- no-connect marks 0 -> 3
Changed lines of the file:
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@@
 (kicad_sch (version 20230121) (generator eeschema)
   (paper "A4")
+  (no_connect (at 130.81 90.17))
+  (no_connect (at 110.49 77.47))
+  (no_connect (at 110.49 90.17))
   (wire (pts (xy 168.91 87.63) (xy 168.91 85.09))
     (stroke (width 0) (type default))
