File: Digit_IN_board/Optopair.kicad_sch (KiCad schematic)
At the start: 42 parts

Commit message: Modify Digit_IN, Motherbord, Step motors
Parts:
- C16, C17, C18, C19: value 0.1uF 100V 0805 -> 0,1uF 100V 0805
- OC2: value IS281- 4 -> IS281- 4 (SOIC-16W)
Changed lines of the file:
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@@
       (effects (font (size 1.27 1.27)) (justify left))
     )
-    (property "Value" "0.1uF 100V 0805" (at 73.66 163.83 90)
+    (property "Value" "0,1uF 100V 0805" (at 73.66 163.83 90)
       (effects (font (size 1.27 1.27)) (justify left))
     )
@@
       (effects (font (size 1.27 1.27)) (justify left))
     )
-    (property "Value" "0.1uF 100V 0805" (at 85.09 163.83 90)
+    (property "Value" "0,1uF 100V 0805" (at 85.09 163.83 90)
       (effects (font (size 1.27 1.27)) (justify left))
     )
@@
       (effects (font (size 1.27 1.27)) (justify left))
     )
-    (property "Value" "0.1uF 100V 0805" (at 73.66 81.28 90)
+    (property "Value" "0,1uF 100V 0805" (at 73.66 81.28 90)
       (effects (font (size 1.27 1.27)) (justify left))
     )
@@
       (effects (font (size 1.27 1.27)))
     )
-    (property "Value" "IS281- 4" (at 139.7 31.75 0)
+    (property "Value" "IS281- 4 (SOIC-16W)" (at 139.7 31.75 0)
       (effects (font (size 1.27 1.27)))
     )
@@
       (effects (font (size 1.27 1.27)) (justify left))
     )
-    (property "Value" "0.1uF 100V 0805" (at 96.52 81.28 90)
+    (property "Value" "0,1uF 100V 0805" (at 96.52 81.28 90)
       (effects (font (size 1.27 1.27)) (justify left))
     )
@@
       (effects (font (size 1.27 1.27)) (justify left))
     )
-    (property "Value" "0.1uF 100V 0805" (at 107.95 163.83 90)
+    (property "Value" "0,1uF 100V 0805" (at 107.95 163.83 90)
       (effects (font (size 1.27 1.27)) (justify left))
     )
@@
       (effects (font (size 1.27 1.27)) (justify left))
     )
-    (property "Value" "0.1uF 100V 0805" (at 85.09 81.28 90)
+    (property "Value" "0,1uF 100V 0805" (at 85.09 81.28 90)
       (effects (font (size 1.27 1.27)) (justify left))
     )
@@
       (effects (font (size 1.27 1.27)) (justify left))
     )
-    (property "Value" "0.1uF 100V 0805" (at 96.52 163.83 90)
+    (property "Value" "0,1uF 100V 0805" (at 96.52 163.83 90)
       (effects (font (size 1.27 1.27)) (justify left))
     )
@@
       (effects (font (size 1.27 1.27)))
     )
-    (property "Value" "IS281- 4" (at 142.24 114.3 0)
+    (property "Value" "IS281- 4 (SOIC-16W)" (at 142.24 114.3 0)
       (effects (font (size 1.27 1.27)))
     )
@@
       (effects (font (size 1.27 1.27)) (justify left))
     )
-    (property "Value" "0.1uF 100V 0805" (at 107.95 81.28 90)
-      (effects (font (size 1.27 1.27)) (justify left))
-    )
+    (property "Value" "0,1uF 100V 0805" (at 107.95 81.28 90)
+      (effects (font (size 1.27 1.27)) (justify left))
+    )

Commit message: Modify DiscretIN Schems and PCB1
Other:
- moved on the sheet: R26
