File: Motherboard/Материнская плата для производства/Материнская плата.kicad_pcb (KiCad board)
At the start: 2 copper layers, 291 x 81 mm, 83 parts, among them J1 SL-10 (L-KLS1-603C-10-S), J10 SL-10 (L-KLS1-603C-10-S), J11 SL-10 (L-KLS1-603C-10-S), J12 SL-10 (L-KLS1-603C-10-S), J13 SL-10 (L-KLS1-603C-10-S), J14 SL-10 (L-KLS1-603C-10-S), J15 SL-10 (L-KLS1-603C-10-S), J16 SL-10 (L-KLS1-603C-10-S), J17 SL-10 (L-KLS1-603C-10-S), J18 SL-10 (L-KLS1-603C-10-S), J19 SL-10 (L-KLS1-603C-10-S), J2 SL-10 (L-KLS1-603C-10-S), J20 SL-10 (L-KLS1-603C-10-S), J21 SL-10 (L-KLS1-603C-10-S), J22 SL-10 (L-KLS1-603C-10-S), J23 SL-10 (L-KLS1-603C-10-S), J24 SL-10 (L-KLS1-603C-10-S), J25 SL-10 (L-KLS1-603C-10-S), J26 DG142V-5.08-02P-14, J27 DG142V-5.08-02P-14, J3 SL-14 (L-KLS1-603C-14-S), J4 SL-10 (L-KLS1-603C-10-S), J5 SL-10 (L-KLS1-603C-10-S), J6 SL-10 (L-KLS1-603C-10-S), J7 SL-10 (L-KLS1-603C-10-S), J8 SL-10 (L-KLS1-603C-10-S), J9 SL-10 (L-KLS1-603C-10-S), Q1 SUM110P06-08L-E3, Q3 SUM110P06-08L-E3, U1 TL431DBZ (sot-23), U2 AM1SS-2403SJZ

Commit message: renew all schems and pcb for production
Parts:
- D1, D10, D2, D3, D4, D5, D6, D7, D8, D9: value SMBJ5.0A -> SMBJ5.0A (SMB)
- D11: value SM6T30A -> SM6T30A (SMB)
- Q1, Q3: value SUM110P06-08L-E3 -> SUM110P06-08L-E3 (TO-263-2)
- R1: value 121 1206 -> 1206-120 Ом±5%-0,25 Вт
- R2: value 242 2512 -> 2512-2,4 кОм±5%-1 Вт
- R3, R7: value 103 0805 -> 0805-10 кОм±5%-0,125 Вт
- R4: value 152 0805 -> 0805-1,5 кОм±5%-0,125 Вт
- R5, R6: value 102 1206 -> 1206-1 кОм±5%-0,25 Вт
- R8: value 201 0805 -> 0805-200 Ом±5%-0,125 Вт
