File: LED_and_photodiode_board/PhotoTransistor.kicad_sch (KiCad schematic)
At the start: 4 parts, among them Q1 PT91-21B/TR7

Commit message: renew schems
Parts:
- C1: value 0.1uF 100V 0805 -> 0,1uF 100V 0805
- Q1: value PT91-21B/TR7 -> PT91-21B/TR7 (1206)
Changed lines of the file:
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@@
       (effects (font (size 1.27 1.27)) (justify left))
     )
-    (property "Value" "0.1uF 100V 0805" (at 133.35 102.87 90)
+    (property "Value" "0,1uF 100V 0805" (at 133.35 102.87 90)
       (effects (font (size 1.27 1.27)) (justify left))
     )
@@
       (effects (font (size 1.27 1.27)) (justify left))
     )
-    (property "Value" "PT91-21B/TR7" (at 119.38 97.79 90)
+    (property "Value" "PT91-21B/TR7 (1206)" (at 119.38 97.79 90)
       (effects (font (size 1.27 1.27)) (justify left))
     )
@@
       (effects (font (size 1.27 1.27)) (justify left))
     )
-    (property "Value" "0.1uF 100V 0805" (at 101.6 86.36 90)
+    (property "Value" "0,1uF 100V 0805" (at 101.6 86.36 90)
       (effects (font (size 1.27 1.27)) (justify left))
     )

Commit message: renew all schems and pcb for production
Parts:
- R9: value 243 0805 -> 0805-24 кОм±5%-0,125 Вт
Changed lines of the file:
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@@
       (effects (font (size 1.27 1.27)) (justify left))
     )
-    (property "Value" "243 0805" (at 116.84 73.66 0)
+    (property "Value" "0805-24 кОм±5%-0,125 Вт" (at 116.84 73.66 0)
       (effects (font (size 1.27 1.27)) (justify left))
     )

Commit message: RENEW ALL BOARDS
Parts:
- R9: value 0805-24 кОм±5%-0,125 Вт -> 0805-51 кОм±5%-0,125 Вт
Changed lines of the file:
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@@
       (effects (font (size 1.27 1.27)) (justify left))
     )
-    (property "Value" "0805-24 кОм±5%-0,125 Вт" (at 116.84 73.66 0)
+    (property "Value" "0805-51 кОм±5%-0,125 Вт" (at 116.84 73.66 0)
       (effects (font (size 1.27 1.27)) (justify left))
     )
