File: Analog_IO_board/Triak.kicad_sch (KiCad schematic)
At the start: 12 parts, among them Q1 DTC114ECA (SOT-23), Q3 BT136X-800E TO-220

Commit message: renew all schems and pcb for production
Parts:
- TP11, TP12: now left out of the parts list
Changed lines of the file:
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@@
   )
   (symbol (lib_id "Connector:TestPoint") (at 101.6 92.71 0) (mirror y) (unit 1)
-    (in_bom yes) (on_board yes) (dnp no)
+    (in_bom no) (on_board yes) (dnp no)
     (property "Reference" "TP11" (at 99.06 88.138 0)
       (effects (font (size 1.27 1.27)) (justify left))
     )
     (property "Value" "TestPoint" (at 99.06 90.678 0)
-      (effects (font (size 1.27 1.27)) (justify left))
+      (effects (font (size 1.27 1.27)) (justify left) hide)
     )
     (property "Footprint" "PCM_4ms_TestPoint:TestPoint_D1" (at 96.52 92.71 0)
@@
   )
   (symbol (lib_id "Connector:TestPoint") (at 187.96 105.41 0) (unit 1)
-    (in_bom yes) (on_board yes) (dnp no) (fields_autoplaced)
+    (in_bom no) (on_board yes) (dnp no) (fields_autoplaced)
     (property "Reference" "TP12" (at 190.5 100.838 0)
       (effects (font (size 1.27 1.27)) (justify left))
     )
     (property "Value" "TestPoint" (at 190.5 103.378 0)
-      (effects (font (size 1.27 1.27)) (justify left))
+      (effects (font (size 1.27 1.27)) (justify left) hide)
     )
     (property "Footprint" "PCM_4ms_TestPoint:TestPoint_D1" (at 193.04 105.41 0)

Commit message: anlog IO pcb and shcems
Parts:
- R12, R13, R14: footprint PCM_4ms_Resistor:R_0805_2012Metric -> PCM_Resistor_SMD_AKL:R_2512_6332Metric

Commit message: qr and analog refresh
Parts:
- R12: value 181 2512 -> 2512-180 Ом±5%-1 Вт
- R13: value 102 2512 -> 2512-1 кОм±5%-1 Вт
- R14: value 510 2512 -> 2512-51 Ом±5%-1 Вт
- R15: value 201 0805 -> 0805-200 Ом±5%-0,125 Вт
Changed lines of the file:
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@@
       (effects (font (size 1.27 1.27)))
     )
-    (property "Value" "201 0805" (at 95.25 78.74 90)
+    (property "Value" "0805-200 Ом±5%-0,125 Вт" (at 95.25 78.74 90)
       (effects (font (size 1.27 1.27)))
     )
@@
       (effects (font (size 1.27 1.27)) (justify right))
     )
-    (property "Value" "510 2512" (at 176.53 82.55 0)
+    (property "Value" "2512-51 Ом±5%-1 Вт" (at 176.53 82.55 0)
       (effects (font (size 1.27 1.27)) (justify right))
     )
@@
       (effects (font (size 1.27 1.27)))
     )
-    (property "Value" "181 2512" (at 123.19 68.58 90)
+    (property "Value" "2512-180 Ом±5%-1 Вт" (at 123.19 68.58 90)
       (effects (font (size 1.27 1.27)))
     )
@@
       (effects (font (size 1.27 1.27)))
     )
-    (property "Value" "102 2512" (at 134.62 68.58 90)
-      (effects (font (size 1.27 1.27)))
-    )
+    (property "Value" "2512-1 кОм±5%-1 Вт" (at 134.62 68.58 90)
+      (effects (font (size 1.27 1.27)))
+    )
