File: QR code/Плата QR.kicad_sch (KiCad schematic)
At the start: 46 parts, among them J1 Prog (PinHeader_2x03_P2.54mm), J10 DG141R-04, J8 Debbag GPIO (PinHeader_01x02_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, J9 DG141R-04, Q1 DTC114ECA (SOT-23), Q2 DTC114ECA (SOT-23), U1 pia141M30 (SOIC-16), U2 ADM3485EARZ-REEL (SOIC-8), U3 STM32G070RBTx (LQFP-64), U4 AM1SS-2403SJZ

Commit message: qr code schems and pcb
Parts:
- added TP19 (x3): TestPoint, PCM_4ms_TestPoint:TestPoint_D1, symbol Connector:TestPoint
Connections:
- net +24V: now also TP19.1
- net +3V3: now also TP19.1
- net GNDA: now also TP19.1
Changed lines of the file:
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@@
   (junction (at 30.48 184.15) (diameter 0) (color 0 0 0 0)
   )
+  (junction (at 248.92 142.24) (diameter 0) (color 0 0 0 0)
+  )
   (junction (at 107.95 20.32) (diameter 0) (color 0 0 0 0)
   )
@@
   (junction (at 80.01 46.99) (diameter 0) (color 0 0 0 0)
   )
+  (junction (at 163.83 156.21) (diameter 0) (color 0 0 0 0)
+  )
   (junction (at 191.77 142.24) (diameter 0) (color 0 0 0 0)
   )
@@
   (junction (at 63.5 176.53) (diameter 0) (color 0 0 0 0)
   )
+  (junction (at 58.42 176.53) (diameter 0) (color 0 0 0 0)
+  )
   (no_connect (at 267.97 95.25))
   (wire (pts (xy 62.23 22.86) (xy 87.63 22.86))
@@
     (stroke (width 0) (type default))
   )
+  (wire (pts (xy 248.92 142.24) (xy 255.27 142.24))
+    (stroke (width 0) (type default))
+  )
   (wire (pts (xy 62.23 26.67) (xy 62.23 30.48))
     (stroke (width 0) (type default))
   )
+  (wire (pts (xy 163.83 156.21) (xy 163.83 151.13))
+    (stroke (width 0) (type default))
+  )
+  (wire (pts (xy 58.42 176.53) (xy 63.5 176.53))
+    (stroke (width 0) (type default))
+  )
   (wire (pts (xy 17.78 184.15) (xy 17.78 186.69))
     (stroke (width 0) (type default))
@@
     (stroke (width 0) (type default))
   )
-  (wire (pts (xy 50.8 176.53) (xy 63.5 176.53))
+  (wire (pts (xy 50.8 176.53) (xy 58.42 176.53))
     (stroke (width 0) (type default))
   )
@@
     (stroke (width 0) (type default))
   )
-  (wire (pts (xy 245.11 142.24) (xy 255.27 142.24))
+  (wire (pts (xy 245.11 142.24) (xy 248.92 142.24))
     (stroke (width 0) (type default))
   )
@@
     )
   )
+  (symbol (lib_id "Connector:TestPoint") (at 163.83 156.21 90) (unit 1)
+    (in_bom no) (on_board yes) (dnp no) (fields_autoplaced)
+    (property "Reference" "TP19" (at 160.528 153.67 90)
+      (effects (font (size 1.27 1.27)))
+    )
+    (property "Value" "TestPoint" (at 161.798 153.67 0)
+      (effects (font (size 1.27 1.27)) (justify left) hide)
+    )
+    (property "Footprint" "PCM_4ms_TestPoint:TestPoint_D1" (at 163.83 151.13 0)
+      (effects (font (size 1.27 1.27)) hide)
+    )
+    (property "Datasheet" "~" (at 163.83 151.13 0)
+      (effects (font (size 1.27 1.27)) hide)
+    )
+    (pin "1")
+    (instances
+      (project "Плата симистров"
+        (path "/271a56a4-fac2-444b-8acf-7cf36bf0ab17"
+          (reference "TP19") (unit 1)
+        )
+      )
+      (project "Плата QR"
+        (path "/5de11a73-9d1a-46ee-891f-a56220952d72"
+          (reference "TP9") (unit 1)
+        )
+      )
+      (project "Плата внешних шаговых двигателей"
+        (path "/7f8f7dc9-8c50-44ed-985c-35a6d8c67be0/0d239b34-7914-40bc-9b83-7e562c30defe"
+          (reference "TP21") (unit 1)
+        )
+        (path "/7f8f7dc9-8c50-44ed-985c-35a6d8c67be0/1f6eaeee-a46e-4730-b225-3a410300814a"
+          (reference "TP5") (unit 1)
+        )
+      )
+    )
+  )
   (symbol (lib_id "Device:C") (at 173.99 43.18 0) (unit 1)
     (in_bom yes) (on_board yes) (dnp no) (fields_autoplaced)
@@
     )
   )
+  (symbol (lib_id "Connector:TestPoint") (at 248.92 142.24 0) (unit 1)
+    (in_bom no) (on_board yes) (dnp no) (fields_autoplaced)
+    (property "Reference" "TP19" (at 251.46 137.668 0)
+      (effects (font (size 1.27 1.27)) (justify left))
+    )
+    (property "Value" "TestPoint" (at 251.46 140.208 0)
+      (effects (font (size 1.27 1.27)) (justify left) hide)
+    )
+    (property "Footprint" "PCM_4ms_TestPoint:TestPoint_D1" (at 254 142.24 0)
+      (effects (font (size 1.27 1.27)) hide)
+    )
+    (property "Datasheet" "~" (at 254 142.24 0)
+      (effects (font (size 1.27 1.27)) hide)
+    )
+    (pin "1")
+    (instances
+      (project "Плата симистров"
+        (path "/271a56a4-fac2-444b-8acf-7cf36bf0ab17"
+          (reference "TP19") (unit 1)
+        )
+      )
+      (project "Плата QR"
+        (path "/5de11a73-9d1a-46ee-891f-a56220952d72"
+          (reference "TP7") (unit 1)
+        )
+      )
+      (project "Плата внешних шаговых двигателей"
+        (path "/7f8f7dc9-8c50-44ed-985c-35a6d8c67be0/0d239b34-7914-40bc-9b83-7e562c30defe"
+          (reference "TP21") (unit 1)
+        )
+        (path "/7f8f7dc9-8c50-44ed-985c-35a6d8c67be0/1f6eaeee-a46e-4730-b225-3a410300814a"
+          (reference "TP5") (unit 1)
+        )
+      )
+    )
+  )
+  (symbol (lib_id "Connector:TestPoint") (at 58.42 176.53 0) (unit 1)
+    (in_bom no) (on_board yes) (dnp no) (fields_autoplaced)
+    (property "Reference" "TP19" (at 60.96 171.958 0)
+      (effects (font (size 1.27 1.27)) (justify left))
+    )
+    (property "Value" "TestPoint" (at 60.96 174.498 0)
+      (effects (font (size 1.27 1.27)) (justify left) hide)
+    )
+    (property "Footprint" "PCM_4ms_TestPoint:TestPoint_D1" (at 63.5 176.53 0)
+      (effects (font (size 1.27 1.27)) hide)
+    )
+    (property "Datasheet" "~" (at 63.5 176.53 0)
+      (effects (font (size 1.27 1.27)) hide)
+    )
+    (pin "1")
+    (instances
+      (project "Плата симистров"
+        (path "/271a56a4-fac2-444b-8acf-7cf36bf0ab17"
+          (reference "TP19") (unit 1)
+        )
+      )
+      (project "Плата QR"
+        (path "/5de11a73-9d1a-46ee-891f-a56220952d72"
+          (reference "TP8") (unit 1)
+        )
+      )
+      (project "Плата внешних шаговых двигателей"
+        (path "/7f8f7dc9-8c50-44ed-985c-35a6d8c67be0/0d239b34-7914-40bc-9b83-7e562c30defe"
+          (reference "TP21") (unit 1)
+        )
+        (path "/7f8f7dc9-8c50-44ed-985c-35a6d8c67be0/1f6eaeee-a46e-4730-b225-3a410300814a"
+          (reference "TP5") (unit 1)
+        )
+      )
+    )
+  )
   (symbol (lib_id "Converter_DCDC:AM1SS-") (at 223.52 152.4 0) (mirror x) (unit 1)
     (in_bom yes) (on_board yes) (dnp no)
@@
     )
   )
-  (symbol (lib_id "PCM_4ms_Power-symbol:GNDA") (at 163.83 151.13 0) (unit 1)
+  (symbol (lib_id "PCM_4ms_Power-symbol:GNDA") (at 163.83 156.21 0) (unit 1)
     (in_bom yes) (on_board yes) (dnp no) (fields_autoplaced)
-    (property "Reference" "#PWR027" (at 163.83 157.48 0)
+    (property "Reference" "#PWR027" (at 163.83 162.56 0)
       (effects (font (size 1.27 1.27)) hide)
     )
-    (property "Value" "GNDA" (at 163.83 156.21 0)
+    (property "Value" "GNDA" (at 163.83 161.29 0)
       (effects (font (size 1.27 1.27)))
     )
-    (property "Footprint" "" (at 163.83 151.13 0)
+    (property "Footprint" "" (at 163.83 156.21 0)
       (effects (font (size 1.27 1.27)) hide)
     )
-    (property "Datasheet" "" (at 163.83 151.13 0)
+    (property "Datasheet" "" (at 163.83 156.21 0)
       (effects (font (size 1.27 1.27)) hide)
     )

Commit message: qr and analog refresh
Parts:
- C13, C2: value 270 pf X7R 1206 2000v 202R18W271KW4E -> 270 pF X7R 1206 2000v 202R18W271KW4E
- C14: value 47uF 63V D10,5 -> 47uF 63V D6.3 H11
- C3, C6, C7: value 0,1uF 50V 0805 -> 0,1uF 100V 0805
- U1: value pia141M30 (SOIC-16) -> PAI141M30 (SOIC-16)
Changed lines of the file:
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@@
       (effects (font (size 1.27 1.27)) (justify left))
     )
-    (property "Value" "0,1uF 50V 0805" (at 189.23 27.94 0)
+    (property "Value" "0,1uF 100V 0805" (at 189.23 27.94 0)
       (effects (font (size 1.27 1.27)) (justify left))
     )
@@
       (effects (font (size 1.27 1.27)))
     )
-    (property "Value" " 270 pf X7R 1206 2000v 202R18W271KW4E" (at 224.79 163.83 90)
+    (property "Value" "270 pF X7R 1206 2000v 202R18W271KW4E" (at 224.79 163.83 90)
       (effects (font (size 1.27 1.27)))
     )
@@
       (effects (font (size 1.27 1.27)) (justify left))
     )
-    (property "Value" "47uF 63V D10,5" (at 64.77 186.69 0)
+    (property "Value" "47uF 63V D6.3 H11" (at 64.77 186.69 0)
       (effects (font (size 1.27 1.27)) (justify left))
     )
@@
       (effects (font (size 1.27 1.27)) (justify left))
     )
-    (property "Value" "0,1uF 50V 0805" (at 237.49 22.86 0)
+    (property "Value" "0,1uF 100V 0805" (at 237.49 22.86 0)
       (effects (font (size 1.27 1.27)) (justify left))
     )
@@
       (effects (font (size 1.27 1.27)))
     )
-    (property "Value" "pia141M30 (SOIC-16)" (at 123.19 59.69 0)
+    (property "Value" "PAI141M30 (SOIC-16)" (at 123.19 59.69 0)
       (effects (font (size 1.27 1.27)))
     )
@@
       (effects (font (size 1.27 1.27)) (justify left))
     )
-    (property "Value" "0,1uF 50V 0805" (at 177.8 44.45 0)
+    (property "Value" "0,1uF 100V 0805" (at 177.8 44.45 0)
       (effects (font (size 1.27 1.27)) (justify left))
     )
@@
       (effects (font (size 1.27 1.27)))
     )
-    (property "Value" " 270 pf X7R 1206 2000v 202R18W271KW4E" (at 124.46 16.51 90)
-      (effects (font (size 1.27 1.27)))
-    )
+    (property "Value" "270 pF X7R 1206 2000v 202R18W271KW4E" (at 124.46 16.51 90)
+      (effects (font (size 1.27 1.27)))
+    )
