File: motherboard/motherboard.kicad_pcb (KiCad board)
At the start: 2 copper layers, 291 x 81 mm, 83 parts, among them J1 SL-10 (L-KLS1-603C-10-S), J10 SL-10 (L-KLS1-603C-10-S), J11 SL-10 (L-KLS1-603C-10-S), J12 SL-10 (L-KLS1-603C-10-S), J13 SL-10 (L-KLS1-603C-10-S), J14 SL-10 (L-KLS1-603C-10-S), J15 SL-10 (L-KLS1-603C-10-S), J16 SL-10 (L-KLS1-603C-10-S), J17 SL-10 (L-KLS1-603C-10-S), J18 SL-10 (L-KLS1-603C-10-S), J19 SL-10 (L-KLS1-603C-10-S), J2 SL-10 (L-KLS1-603C-10-S), J20 SL-10 (L-KLS1-603C-10-S), J21 SL-10 (L-KLS1-603C-10-S), J22 SL-10 (L-KLS1-603C-10-S), J23 SL-10 (L-KLS1-603C-10-S), J24 SL-10 (L-KLS1-603C-10-S), J25 SL-10 (L-KLS1-603C-10-S), J26 DG142V-5.08-02P-14, J27 DG142V-5.08-02P-14, J3 SL-14 (L-KLS1-603C-14-S), J4 SL-10 (L-KLS1-603C-10-S), J5 SL-10 (L-KLS1-603C-10-S), J6 SL-10 (L-KLS1-603C-10-S), J7 SL-10 (L-KLS1-603C-10-S), J8 SL-10 (L-KLS1-603C-10-S), J9 SL-10 (L-KLS1-603C-10-S), Q1 SUM110P06-08L-E3 (TO-263-2), Q3 SUM110P06-08L-E3 (TO-263-2), U1 TL431DBZ (sot-23), U2 AM1SS-2403SJZ

Commit message: DC, contr, mb, step v2
Parts:
- added G***: LOGO, Symbol:PB_LOGO, F.Cu at (5.50, 66.5)
- added J28: PinHeader_1x02_P2.54mm (Contr +24V), Connector_PinHeader_2.54mm:PinHeader_1x02_P2.54mm_Vertical, F.Cu at (290.0, 79.0)
- added J29: PinHeader_1x04_P2.54mm (RS485), Connector_PinHeader_2.54mm:PinHeader_1x04_P2.54mm_Vertical, F.Cu at (288.5, 37.0)
- added J30: PinHeader_2x07_P2.54mm (RTS), Connector_PinHeader_2.54mm:PinHeader_2x07_P2.54mm_Vertical, F.Cu at (289.0, 55.0)
- D11: value SM6T30A (SMB) -> SM6T30CA (SMB)
- F1, F2: value Fuse 10A ZH266 (2 клипсы) -> Fuse 5A ZH266 (2 клипсы)
Routing:
- net /A: track 271.5 -> 301.0 mm
- net /B: track 271.1 -> 297.8 mm
- net GNDA: track 21.9 -> 38.6 mm
- net +24V: track 626.7 -> 643.4 mm
- net /RTS9: track 228.1 -> 239.1 mm
- net /RTS5: track 130.0 -> 140.9 mm
- net /RTS3: track 80.9 -> 91.9 mm
- net /RTS1: track 31.9 -> 42.8 mm
- net /RTS7: track 179.0 -> 190.0 mm
- net /RTS11: track 277.1 -> 288.1 mm
- net /RTS10: track 257.2 -> 265.6 mm
- net /RTS8: track 208.1 -> 216.5 mm
- net /RTS6: track 159.1 -> 167.5 mm
- net /RTS4: track 110.0 -> 118.4 mm
- net /RTS2: track 60.9 -> 69.4 mm
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Other:
- board text added: "+"
- board text added: "1"
- board text added: "2"
- board text added: "A"
- board text added: "B"
- board text added: "G"
- board text added: "t01 v02 a"

Commit message: DC, contr, mb, digit in v2.1
Parts:
- moved D12 2.65 mm to (196.2, 97.5)
- moved RV1 2.22 mm to (47.9, 42.1), turned to 0 degrees
- moved C3 1.49 mm to (32.0, 64.0), turned to 0 degrees
- moved R7 1.41 mm to (224.5, 71.0), turned to 180 degrees
- moved RV5 1.30 mm to (241.7, 43.3)
- moved R3 1.00 mm to (239.0, 80.5)
- moved RV2 0.98 mm to (96.1, 41.9), turned to 0 degrees
- moved RV3 0.77 mm to (145.6, 42.2), turned to 0 degrees
- moved RV4 0.55 mm to (193.3, 42.0), turned to 0 degrees
- moved C4 0.52 mm to (31.8, 81.5)
Connections:
- H1 pad 1: GND1 -> unconnected-(H1-Pad1)
- H10 pad 1: GNDA -> unconnected-(H10-Pad1)
- H11 pad 1: GNDA -> unconnected-(H11-Pad1)
- H12 pad 1: GNDA -> unconnected-(H12-Pad1)
- H13 pad 1: GND1 -> unconnected-(H13-Pad1)
- H14 pad 1: GNDA -> unconnected-(H14-Pad1)
- H2 pad 1: GND1 -> unconnected-(H2-Pad1)
- H3 pad 1: GND1 -> unconnected-(H3-Pad1)
- H4 pad 1: GND1 -> unconnected-(H4-Pad1)
- H5 pad 1: GND1 -> unconnected-(H5-Pad1)
- H6 pad 1: GND1 -> unconnected-(H6-Pad1)
- H7 pad 1: GNDA -> unconnected-(H7-Pad1)
- H8 pad 1: GNDA -> unconnected-(H8-Pad1)
- H9 pad 1: GNDA -> unconnected-(H9-Pad1)
Routing:
- net /A: track 301.0 -> 356.6 mm
- net /B: track 297.8 -> 348.9 mm
- net Net-(D11-A2): track 59.7 -> 70.5 mm
- net Net-(Q1-G): track 9.59 -> 17.8 mm
- net Net-(D14-K): track 3.00 -> 5.89 mm
- net Net-(U1-REF): track 4.23 -> 6.86 mm
- net GND1: track 265.6 -> 263.1 mm, vias 153 -> 151
- net /+3.3VRS485: track 349.1 -> 347.5 mm
- net Net-(D13-K): track 48.5 -> 49.5 mm
- net Net-(D12-K): track 3.10 -> 3.99 mm
- net Net-(D11-A1): track 54.4 -> 54.9 mm

Commit message: Triak v2.1
Routing:
- net /B: track 348.9 -> 356.3 mm
- net /A: track 356.6 -> 363.6 mm

Commit message: mother  убраны ловушки
Routing:
- net Net-(U1-REF): track 6.86 -> 0.00 mm
- net GNDA: track 38.6 -> 34.2 mm
- added copper zone on B.Cu, net Net-(U1-REF)

Commit message: motherboard установлены тестовые площадки
Parts:
- added TP1: TestPoint, PCM_4ms_TestPoint:TestPoint_D1, B.Cu at (259.8, 38.1)
- added TP10: TestPoint, PCM_4ms_TestPoint:TestPoint_D1, B.Cu at (270.7, 53.8)
- added TP11: TestPoint, PCM_4ms_TestPoint:TestPoint_D1, B.Cu at (270.8, 56.3)
- added TP12: TestPoint, PCM_4ms_TestPoint:TestPoint_D1, B.Cu at (270.7, 58.9)
- added TP13: TestPoint, PCM_4ms_TestPoint:TestPoint_D1, B.Cu at (270.6, 61.4)
- added TP14: TestPoint, PCM_4ms_TestPoint:TestPoint_D1, B.Cu at (193.1, 91.3)
- added TP15: TestPoint, PCM_4ms_TestPoint:TestPoint_D1, B.Cu at (30.7, 64.1)
- added TP16: TestPoint, PCM_4ms_TestPoint:TestPoint_D1, B.Cu at (196.1, 94.9)
- added TP17: TestPoint, PCM_4ms_TestPoint:TestPoint_D1, B.Cu at (268.7, 39.9)
- added TP18: TestPoint, PCM_4ms_TestPoint:TestPoint_D1, B.Cu at (238.9, 84.1)
- added TP19: TestPoint, PCM_4ms_TestPoint:TestPoint_D1, B.Cu at (232.4, 76.4)
- added TP2: TestPoint, PCM_4ms_TestPoint:TestPoint_D1, B.Cu at (259.7, 40.6)
- added TP20: TestPoint, PCM_4ms_TestPoint:TestPoint_D1, B.Cu at (244.9, 85.8)
- added TP3: TestPoint, PCM_4ms_TestPoint:TestPoint_D1, B.Cu at (276.9, 52.5)
- added TP4: TestPoint, PCM_4ms_TestPoint:TestPoint_D1, B.Cu at (276.8, 55.0)
- added TP5: TestPoint, PCM_4ms_TestPoint:TestPoint_D1, B.Cu at (276.8, 57.7)
- added TP6: TestPoint, PCM_4ms_TestPoint:TestPoint_D1, B.Cu at (276.7, 60.1)
- added TP7: TestPoint, PCM_4ms_TestPoint:TestPoint_D1, B.Cu at (276.7, 62.7)
- added TP8: TestPoint, PCM_4ms_TestPoint:TestPoint_D1, B.Cu at (276.7, 65.2)
- added TP9: TestPoint, PCM_4ms_TestPoint:TestPoint_D1, B.Cu at (270.9, 50.5)
Routing:
- net Net-(D11-A2): track 70.5 -> 76.0 mm
- net Net-(Q1-S): track 33.2 -> 38.5 mm, vias 0 -> 1
- net /B: track 356.1 -> 359.7 mm
- net /A: track 363.7 -> 367.3 mm
- net /+3.3VRS485: track 347.5 -> 350.3 mm
- net /RTS9: track 239.1 -> 241.4 mm
- net /RTS7: track 190.0 -> 192.3 mm
- net /RTS11: track 288.1 -> 290.4 mm
- net /RTS5: track 140.9 -> 143.2 mm
- net /RTS3: track 91.9 -> 94.1 mm
- net /RTS1: track 42.8 -> 45.0 mm
- net Net-(D13-K): track 49.0 -> 50.6 mm
