File: manipulator_attachment/Magnit.kicad_sch (KiCad schematic)
At the start: 4 parts, among them Q3 FDN5630

Commit message: DC, contr, mb, digit in v2.1
Parts:
- R7: footprint PCM_Resistor_SMD_AKL:R_0603_1608Metric -> Resistor_SMD:R_0603_1608Metric
Changed lines of the file:
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@@
       (effects (font (size 1.27 1.27)))
     )
-    (property "Footprint" "PCM_Resistor_SMD_AKL:R_0603_1608Metric" (at 90.17 95.758 90)
+    (property "Footprint" "Resistor_SMD:R_0603_1608Metric" (at 90.17 95.758 90)
       (effects (font (size 1.27 1.27)) hide)
     )
@@
     (pin "1")
     (instances
-      (project "Плата управления Культи"
+      (project "manipulator_attachment"
         (path "/3077e151-2eda-4625-b5d8-67761d2c8260/5efd83d5-7b96-4f3a-b42e-52d434a47456"
           (reference "R7") (unit 1)
@@
     (pin "2")
     (instances
-      (project "Плата управления Культи"
+      (project "manipulator_attachment"
         (path "/3077e151-2eda-4625-b5d8-67761d2c8260/5efd83d5-7b96-4f3a-b42e-52d434a47456"
           (reference "D5") (unit 1)
@@
     (pin "1")
     (instances
-      (project "Плата управления Культи"
+      (project "manipulator_attachment"
         (path "/3077e151-2eda-4625-b5d8-67761d2c8260/5efd83d5-7b96-4f3a-b42e-52d434a47456"
           (reference "C15") (unit 1)
@@
     (pin "3")
     (instances
-      (project "Плата управления Культи"
+      (project "manipulator_attachment"
         (path "/3077e151-2eda-4625-b5d8-67761d2c8260/5efd83d5-7b96-4f3a-b42e-52d434a47456"
           (reference "Q3") (unit 1)

Commit message: manipulator 1.0
Parts:
- renumbered D5 to D7, R7 to R9
Changed lines of the file:
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@@
   (symbol (lib_id "Device:R") (at 90.17 93.98 90) (unit 1)
     (in_bom yes) (on_board yes) (dnp no) (fields_autoplaced)
-    (property "Reference" "R7" (at 90.17 87.63 90)
+    (property "Reference" "R9" (at 90.17 87.63 90)
       (effects (font (size 1.27 1.27)))
     )
@@
       (project "manipulator_attachment"
         (path "/3077e151-2eda-4625-b5d8-67761d2c8260/5efd83d5-7b96-4f3a-b42e-52d434a47456"
-          (reference "R7") (unit 1)
+          (reference "R9") (unit 1)
         )
       )
@@
   (symbol (lib_id "PCM_Diode_Schottky_AKL:SS16") (at 109.22 71.12 270) (mirror x) (unit 1)
     (in_bom yes) (on_board yes) (dnp no) (fields_autoplaced)
-    (property "Reference" "D5" (at 106.68 69.5325 90)
+    (property "Reference" "D7" (at 106.68 69.5325 90)
       (effects (font (size 1.27 1.27)) (justify right))
     )
@@
       (project "manipulator_attachment"
         (path "/3077e151-2eda-4625-b5d8-67761d2c8260/5efd83d5-7b96-4f3a-b42e-52d434a47456"
-          (reference "D5") (unit 1)
+          (reference "D7") (unit 1)
         )
       )

Commit message: manipulator углы и терминатор
Parts:
- Q3: footprint PCM_Package_TO_SOT_SMD_AKL:SOT-23 -> Package_TO_SOT_SMD:SOT-23
