File: dc_motor_board/PumpV2.kicad_sch (KiCad schematic)
At the start: 48 parts, among them J4 DG142R-5.08-02P-14 OUT, Q4 BTN8962TA, Q5 BTN8962TA, U6 PAI162M30 (SOIC-16)

Commit message: fix dc board issues before manufacturing
Parts:
- C38: footprint PCM_Capacitor_THT_AKL:C_Radial_D10.0mm_H16.0mm_P5.00mm -> PCM_Capacitor_THT_AKL:CP_Radial_D10.0mm_P5.00mm
- C5: renamed from C28; value 0,1uF 50V 0603 -> 0,1uF 100V 0603
- C5: renamed from C35; value 0,1uF 100V 0805 -> 0,1uF 100V 0603; footprint PCM_Capacitor_SMD_AKL:C_0805_2012Metric_Pad1.15x1.40mm -> Capacitor_SMD:C_0603_1608Metric_Pad1.08x0.95mm_HandSolder
- C5: renamed from C15; value 0,1uF 50V 0603 -> 0,1uF 100V 0603
- C5: renamed from C22; value 0,1uF 100V 0805 -> 0,1uF 100V 0603; footprint PCM_Capacitor_SMD_AKL:C_0805_2012Metric_Pad1.15x1.40mm -> Capacitor_SMD:C_0603_1608Metric_Pad1.08x0.95mm_HandSolder
- C9: renamed from C31; value 0,1uF 100V 0805 -> 0,1uF 100V 0603; footprint PCM_Capacitor_SMD_AKL:C_0805_2012Metric_Pad1.15x1.40mm -> Capacitor_SMD:C_0603_1608Metric_Pad1.08x0.95mm_HandSolder
- C9: renamed from C30; value 0,1uF 100V 0805 -> 0,1uF 100V 0603; footprint PCM_Capacitor_SMD_AKL:C_0805_2012Metric_Pad1.15x1.40mm -> Capacitor_SMD:C_0603_1608Metric_Pad1.08x0.95mm_HandSolder
- Q4, Q5: value BTN8962TA -> BTN8962TA (TO-263-7)
- renumbered C45 to C2, TP33 to TP1, TP31 to TP1, TP17 to TP1, TP25 to TP1, TP37 to TP1, TP19 to TP1, TP21 to TP1, TP29 to TP1, TP13 to TP1, TP27 to TP1, TP39 to TP1, TP15 to TP1, TP23 to TP1, TP11 to TP1

Commit message: DC, contr, mb, digit in v2.1
Parts:
- C5, C9: footprint Capacitor_SMD:C_0603_1608Metric_Pad1.08x0.95mm_HandSolder -> Capacitor_SMD:C_0603_1608Metric
- R22, R23, R24, R25, R26, R27, R28, R29, R30, R31, R32, R33: footprint PCM_Resistor_SMD_AKL:R_0603_1608Metric_Pad1.05x0.95mm_HandSolder -> Resistor_SMD:R_0603_1608Metric

Commit message: controller  убраны ловушки
Parts:
- C42: renamed from C38; footprint PCM_Capacitor_THT_AKL:CP_Radial_D10.0mm_P5.00mm -> Capacitor_THT:CP_Radial_D10.0mm_P5.00mm
- C45: renamed from C2; footprint PCM_Capacitor_SMD_Handsoldering_AKL:C_1210_3225Metric_Pad1.42x2.65mm -> Capacitor_SMD:C_1210_3225Metric
- D10, D12, D6, D8: symbol PCM_Diode_Schottky_AKL:STPS2H100A -> Device:D_Schottky
- TP12, TP14, TP16, TP18, TP20, TP22, TP24, TP26, TP28, TP30, TP32, TP34, TP38, TP40: renamed from TP1; footprint PCM_4ms_TestPoint:TestPoint_D1 -> TestPoint:TestPoint_Pad_D1.0mm
- U6: symbol Isolator:π162M3x -> Isolator 7:π162M3x
- renumbered C5 to C16, C5 to C23, C9 to C30, C9 to C31, C5 to C34, C5 to C41

Commit message: update schemas
Parts:
- renumbered C16 to C15, C29 to C17, C30 to C18, C31 to C19, C32 to C20, C33 to C21, C23 to C22, C36 to C24, C37 to C25, C45 to C26, C46 to C27, C34 to C28, C41 to C35, C42 to C38, D12 to D11, D6 to D5, D8 to D7, D10 to D9, J4 to J3, Q4 to Q6, Q5 to Q7, R22 to R10, R23 to R11, R24 to R12, R25 to R13, R26 to R14, R27 to R15, R28 to R16, R29 to R17, R30 to R18, R31 to R19, R32 to R20, R33 to R21, TP12 to TP11, TP14 to TP13, TP16 to TP15, TP18 to TP17, TP20 to TP19, TP22 to TP21, TP24 to TP23, TP26 to TP25, TP28 to TP27, TP30 to TP29, TP32 to TP31, TP34 to TP33, TP38 to TP37, TP40 to TP39, U6 to U5
