File: dc_motor_board/Supply_Voltage_5V.kicad_sch (KiCad schematic)
At the start: 5 parts, among them U7 L78L05 (SOT89-3)

Commit message: fix dc board issues before manufacturing
Parts:
- C40: value 0,1uF 50V 0603 -> 0,1uF 100V 0603
- renumbered R34 to R26

Commit message: DC, contr, mb, digit in v2.1
Parts:
- C40: footprint Capacitor_SMD:C_0603_1608Metric_Pad1.08x0.95mm_HandSolder -> Capacitor_SMD:C_0603_1608Metric
Changed lines of the file:
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@@
     (pin "2")
     (instances
-      (project "Плата насосов"
+      (project "dc_motor_board"
         (path "/7f8f7dc9-8c50-44ed-985c-35a6d8c67be0"
           (reference "R26") (unit 1)
@@
     (pin "2")
     (instances
-      (project "Плата насосов"
+      (project "dc_motor_board"
         (path "/7f8f7dc9-8c50-44ed-985c-35a6d8c67be0/86973487-7b27-4609-9d49-a37377210aac"
           (reference "U7") (unit 1)
@@
     (pin "1")
     (instances
-      (project "Плата насосов"
+      (project "dc_motor_board"
         (path "/7f8f7dc9-8c50-44ed-985c-35a6d8c67be0/86973487-7b27-4609-9d49-a37377210aac"
           (reference "TP1") (unit 1)
@@
     (pin "2")
     (instances
-      (project "Плата насосов"
+      (project "dc_motor_board"
         (path "/7f8f7dc9-8c50-44ed-985c-35a6d8c67be0/86973487-7b27-4609-9d49-a37377210aac"
           (reference "C39") (unit 1)
@@
       (effects (font (size 1.27 1.27)) (justify left))
     )
-    (property "Footprint" "Capacitor_SMD:C_0603_1608Metric_Pad1.08x0.95mm_HandSolder" (at 133.0452 113.03 0)
+    (property "Footprint" "Capacitor_SMD:C_0603_1608Metric" (at 133.0452 113.03 0)
       (effects (font (size 1.27 1.27)) hide)
     )
@@
     (pin "2")
     (instances
-      (project "Плата насосов"
+      (project "dc_motor_board"
         (path "/7f8f7dc9-8c50-44ed-985c-35a6d8c67be0/86973487-7b27-4609-9d49-a37377210aac"
           (reference "C40") (unit 1)

Commit message: controller  убраны ловушки
Parts:
- R34: renamed from R26; footprint PCM_Resistor_SMD_AKL:R_1206_3216Metric_Pad1.42x1.75mm_HandSolder -> Resistor_SMD:R_1206_3216Metric
- TP1: footprint PCM_4ms_TestPoint:TestPoint_D1 -> TestPoint:TestPoint_Pad_D1.0mm
