File: digit_in_board/DiscretOut.kicad_sch (KiCad schematic)
At the start: 107 parts, among them J10 DG142R-5.08-02P-14, J4 DG141R-02, J5 DG141R-02, J6 DG141R-02, J7 DG141R-02, J8 DG141R-02, J9 DG141R-02, Q2 IRFR5305 (TO-252-2), U10 PAI162M30 (SOIC-16), U5 BTS5215 (DSO-12-9), U6 PAI162M30 (SOIC-16), U7 BTS5215, U8 PAI162M30 (SOIC-16), U9 BTS5215

Commit message: digit_in v2
Parts:
- added TP1: ~, PCM_4ms_TestPoint:TestPoint_D1, symbol Connector:TestPoint
- C14: renamed from C22; value 47uF 63V D10,5 -> 47uF 63V D6.3 H11
- C15: renamed from C23; value 0,1uF 100V 0805 -> 0,1uF 100V 0603; footprint PCM_Capacitor_SMD_AKL:C_0805_2012Metric_Pad1.18x1.45mm_HandSolder -> Capacitor_SMD:C_0603_1608Metric
- C9: renamed from C21; footprint PCM_Capacitor_SMD_AKL:C_0603_1608Metric_Pad1.08x0.95mm_HandSolder -> Capacitor_SMD:C_0603_1608Metric
- C9: renamed from C20; footprint PCM_Capacitor_SMD_AKL:C_0603_1608Metric_Pad1.08x0.95mm_HandSolder -> Capacitor_SMD:C_0603_1608Metric
- C9: renamed from C37; value 0,1uF 100V 0805 -> 0,1uF 100V 0603; footprint PCM_Capacitor_SMD_AKL:C_0805_2012Metric_Pad1.18x1.45mm_HandSolder -> Capacitor_SMD:C_0603_1608Metric; now not fitted; now left out of the parts list
- C9: renamed from C19; footprint PCM_Capacitor_SMD_AKL:C_0603_1608Metric_Pad1.08x0.95mm_HandSolder -> Capacitor_SMD:C_0603_1608Metric
- C9: renamed from C38; value 0,1uF 100V 0805 -> 0,1uF 100V 0603; footprint PCM_Capacitor_SMD_AKL:C_0805_2012Metric_Pad1.18x1.45mm_HandSolder -> Capacitor_SMD:C_0603_1608Metric; now not fitted; now left out of the parts list
- C9: renamed from C39; value 0,1uF 100V 0805 -> 0,1uF 100V 0603; footprint PCM_Capacitor_SMD_AKL:C_0805_2012Metric_Pad1.18x1.45mm_HandSolder -> Capacitor_SMD:C_0603_1608Metric; now not fitted; now left out of the parts list
- C9: renamed from C18; footprint PCM_Capacitor_SMD_AKL:C_0603_1608Metric_Pad1.08x0.95mm_HandSolder -> Capacitor_SMD:C_0603_1608Metric
- C9: renamed from C40; value 0,1uF 100V 0805 -> 0,1uF 100V 0603; footprint PCM_Capacitor_SMD_AKL:C_0805_2012Metric_Pad1.18x1.45mm_HandSolder -> Capacitor_SMD:C_0603_1608Metric; now not fitted; now left out of the parts list
- C9: renamed from C16; footprint PCM_Capacitor_SMD_AKL:C_0603_1608Metric_Pad1.08x0.95mm_HandSolder -> Capacitor_SMD:C_0603_1608Metric
- C9: renamed from C36; value 0,1uF 100V 0805 -> 0,1uF 100V 0603; footprint PCM_Capacitor_SMD_AKL:C_0805_2012Metric_Pad1.18x1.45mm_HandSolder -> Capacitor_SMD:C_0603_1608Metric; now not fitted; now left out of the parts list
- C9: renamed from C35; value 0,1uF 100V 0805 -> 0,1uF 100V 0603; footprint PCM_Capacitor_SMD_AKL:C_0805_2012Metric_Pad1.18x1.45mm_HandSolder -> Capacitor_SMD:C_0603_1608Metric; now not fitted; now left out of the parts list
- C9: renamed from C17; footprint PCM_Capacitor_SMD_AKL:C_0603_1608Metric_Pad1.08x0.95mm_HandSolder -> Capacitor_SMD:C_0603_1608Metric
- D3: renamed from D9; value SM6T30A (SMB) -> SM6T30СA (SMB)
- J9: value DG141R-02 -> DG141R-2.54-02P-14-00A(H)
- J9: renamed from J5; value DG141R-02 -> DG141R-2.54-02P-14-00A(H)
- J9: renamed from J7; value DG141R-02 -> DG141R-2.54-02P-14-00A(H)
- J9: renamed from J4; value DG141R-02 -> DG141R-2.54-02P-14-00A(H)
- J9: renamed from J8; value DG141R-02 -> DG141R-2.54-02P-14-00A(H)
- J9: renamed from J6; value DG141R-02 -> DG141R-2.54-02P-14-00A(H)
- Q2: value IRFR5305 (TO-252-2) -> WMO80P06TS (TO-252-2)
- R10, R11, R12, R13, R14, R15, R16, R17, R18, R19, R20, R41, R42, R43, R44, R45, R46, R47, R48, R49, R50, R51, R52, R9: footprint PCM_Resistor_SMD_AKL:R_0603_1608Metric_Pad0.98x0.95mm_HandSolder -> Resistor_SMD:R_0603_1608Metric
- R7: footprint PCM_Resistor_SMD_AKL:R_0805_2012Metric_Pad1.20x1.40mm_HandSolder -> PCM_4ms_Resistor:R_0805_2012Metric
- renumbered TP20 to TP1, TP5 to TP1, TP26 to TP1, TP14 to TP1, TP40 to TP1, TP25 to TP1, TP3 to TP1, TP21 to TP1, TP33 to TP1, TP39 to TP1, TP24 to TP1, TP6 to TP1, TP9 to TP1, TP27 to TP1, TP34 to TP1, TP19 to TP1, TP13 to TP1, TP16 to TP1, TP22 to TP1, TP44 to TP1, TP4 to TP1, TP31 to TP1, TP45 to TP1, TP12 to TP1, TP36 to TP1, TP11 to TP1, TP30 to TP1, TP17 to TP1, TP7 to TP1, TP38 to TP1, TP32 to TP1, TP10 to TP1, TP41 to TP1, TP42 to TP1, TP15 to TP1, TP35 to TP1, TP23 to TP1, TP28 to TP1, TP8 to TP1, TP37 to TP1, TP43 to TP1, TP18 to TP1, TP29 to TP1, TP2 to TP1
Connections:
- net GND2: now also TP1.1
- net +3V3 renamed +3.3V

Commit message: update schemas
Parts:
- U7, U9: value BTS5215 -> BTS5215 (DSO-12-9)
- renumbered C9 to C16, C9 to C17, C9 to C18, C9 to C19, C9 to C20, C9 to C21, C14 to C22, C15 to C23, C9 to C35, C9 to C36, C9 to C37, C9 to C38, C9 to C39, C9 to C40, D3 to D9, TP1 to G2, J9 to J4, J9 to J5, J9 to J6, J9 to J7, J9 to J8, TP1 to TP10, TP1 to TP11, TP1 to TP12, TP1 to TP13, TP1 to TP14, TP1 to TP15, TP1 to TP16, TP1 to TP17, TP1 to TP18, TP1 to TP19, TP1 to TP2, TP1 to TP20, TP1 to TP21, TP1 to TP22, TP1 to TP23, TP1 to TP24, TP1 to TP25, TP1 to TP26, TP1 to TP27, TP1 to TP28, TP1 to TP29, TP1 to TP3, TP1 to TP30, TP1 to TP31, TP1 to TP32, TP1 to TP33, TP1 to TP34, TP1 to TP35, TP1 to TP36, TP1 to TP37, TP1 to TP38, TP1 to TP39, TP1 to TP4, TP1 to TP40, TP1 to TP41, TP1 to TP42, TP1 to TP43, TP1 to TP44, TP1 to TP45, TP1 to TP5, TP1 to TP6, TP1 to TP7, TP1 to TP8, TP1 to TP9
