File: digit_in_board/Supply_Voltage_5V.kicad_sch (KiCad schematic)
At the start: 6 parts, among them U11 L78L05 (SOT89-3)

Commit message: digit_in v2
Parts:
- C25: footprint PCM_Capacitor_SMD_AKL:C_0603_1608Metric_Pad1.08x0.95mm_HandSolder -> Capacitor_SMD:C_0603_1608Metric
- renumbered R22 to R26, R53 to R26

Commit message: update schemas
Parts:
- renumbered R26 to R22, R26 to R53
