File: digit_in_board/digit_in_board.kicad_pcb (KiCad board)
At the start: 2 copper layers, 91.6 x 64.5 mm, 221 parts, among them J10 DG142R-5.08-02P-14, J11 DS1013-01-10RSiB-B (1), J12 DS0, J13 DS0, J2 PLL-10 (Prog), J4 DG141R-2.54-02P-14-00A(H), J5 DG141R-2.54-02P-14-00A(H), J6 DG141R-2.54-02P-14-00A(H), J7 DG141R-2.54-02P-14-00A(H), J8 DG141R-2.54-02P-14-00A(H)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

Commit message: manipulator ловушки
Parts:
- moved TP20 0.32 mm to (130.1, 104.1)
Routing:
- net GND2: track 67.6 -> 64.5 mm
- net +24V: track 19.6 -> 21.5 mm
- net Net-(RS2-Pin_2): track 23.4 -> 22.7 mm

Commit message: digit in test point
Parts:
- TP1, TP46, TP47, TP48, TP49, TP50, TP51, TP52, TP53: moved to B.Cu
- moved TP46 13.8 mm to (123.7, 116.9), turned to 180 degrees
- moved TP47 10.4 mm to (121.4, 116.8), turned to 180 degrees
- moved TP52 9.45 mm to (120.1, 104.9), turned to 180 degrees
- moved TP48 8.22 mm to (117.7, 113.9), turned to 180 degrees
- moved TP50 8.04 mm to (117.7, 111.5), turned to 180 degrees
- moved TP49 6.58 mm to (119.3, 113.3), turned to 180 degrees
- moved TP53 2.02 mm to (117.4, 103.1), turned to 180 degrees
- moved TP51 0.36 mm to (117.4, 104.7), turned to 180 degrees
Routing:
- net GNDD: track 124.4 -> 128.5 mm, vias 48 -> 50
- net /D1: track 27.5 -> 29.7 mm, vias 0 -> 1
- net /D0: track 30.3 -> 32.3 mm, vias 0 -> 1
- net /D7: track 21.7 -> 23.0 mm, vias 0 -> 1
- net +5V: track 77.7 -> 78.8 mm, vias 3 -> 4
- net /D2: track 24.6 -> 25.7 mm, vias 0 -> 1
- net /D6: track 22.7 -> 23.4 mm, vias 0 -> 1
- net /D4: track 23.9 -> 23.3 mm, vias 0 -> 1
- net /D5: track 23.7 -> 24.0 mm, vias 0 -> 1
- net /D3: track 24.4 -> 24.5 mm, vias 0 -> 1

Commit message: update schemas
Parts:
- F1: value 045201.5MRL -> 0451.5MRL (0.5 А)
- J12: value DS0 -> PinHeader_1x03_P2.54mm (DS0)
- J13: value DS0 -> PinHeader_1x03_P2.54mm (DS1)
- U7, U9: value BTS5215 -> BTS5215 (DSO-12-9)
- moved G*** 0.22 mm to (177.9, 74.8)
Routing:
- net GND2: track 64.5 -> 69.0 mm
Other:
- board text added: "PizzaBot inc."
