File: digit_in_board/digit_in_board.kicad_sch (KiCad schematic)
At the start: 46 parts, among them J1 DebugUSART (PinHeader_01x03_P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, J2 Prog (PinHeader_2x03_P2.54mm), J3 Debug GPIO (PinHeader_01x02_P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, Q1 DTC114ECA (SOT-23), Q2 DTC114ECA (SOT-23), U1 PAI141M30 (SOIC-16), U2 ADM3485EARZ-REEL (SOIC-8), U3 STM32G070RBTx (LQFP-64), U4 AM1SS-2403SJZ

Commit message: digit_in v2
Parts:
- removed J1: DebugUSART (PinHeader_01x03_P2.54mm), Connector_PinHeader_2.54mm:PinHeader_1x03_P2.54mm_Vertical, symbol Connector:Conn_01x03_Pin
- removed J2: Prog (PinHeader_2x03_P2.54mm), Connector_PinHeader_2.54mm:PinHeader_2x03_P2.54mm_Vertical, symbol Connector_Generic:Conn_02x03_Odd_Even
- removed J3: Debug GPIO (PinHeader_01x02_P2.54mm), Connector_PinHeader_2.54mm:PinHeader_1x02_P2.54mm_Vertical, symbol Connector:Conn_01x02_Pin
- added C41, C42: 20pF 50V 0603, Capacitor_SMD:C_0603_1608Metric, symbol Device:C
- added J2: PLL-10 (Prog), Connector_PinHeader_1.27mm:PinHeader_1x10_P1.27mm_Vertical, symbol Connector:Conn_01x10_Pin
- added TP1 (x4): ~, PCM_4ms_TestPoint:TestPoint_D1, symbol Connector:TestPoint
- added Y1: Crystal_3225 8MHz, PCM_Crystal_AKL:Crystal_SMD_3225-4Pin_3.2x2.5mm, symbol Device:Crystal_GND24
- C14: value 47uF 63V D10,5 -> 47uF 63V D6.3 H11
- C15, C3, C5, C6, C7, C8, C9: value 0,1uF 100V 0805 -> 0,1uF 100V 0603; footprint PCM_Capacitor_SMD_AKL:C_0805_2012Metric_Pad1.18x1.45mm_HandSolder -> Capacitor_SMD:C_0603_1608Metric
- R4, R8: value 0805-150 Ом±5%-0,125 Вт -> 0603-150 Ом±5%-0,062 Вт; footprint PCM_4ms_Resistor:R_0805_2012Metric -> PCM_4ms_Resistor:R_0603
- renumbered TP65 to TP1, TP67 to TP1, TP64 to TP1, TP63 to TP1, TP62 to TP1, TP66 to TP1
Connections:
- net +3V3: now also J2.1 (Pin_1), TP1.1
- net GND1: now also TP1.1
- net GNDA: now also TP1.1
- net GNDD: now also C41.2, C42.2, J2.6 (Pin_6), TP1.1, Y1.2, Y1.4
- net GPIO1: now also J2.9 (Pin_9)
- net GPIO2: now also J2.10 (Pin_10)
- net NRST: now also J2.5 (Pin_5)
- net SWCLK: now also J2.3 (Pin_3)
- net SWDIO: now also J2.4 (Pin_4)
- net UART_RX: now also J2.8 (Pin_8)
- net UART_TX: now also J2.7 (Pin_7)
- net OSC_IN: now reaches U3.10 (PF0)
- net OSC_IN: now also C41.1, Y1.1
- net OSC_OUT: now reaches U3.11 (PF1)
- net OSC_OUT: now also C42.1, Y1.3
- net UART_DE: no longer names the net of U3.39 (PC7)
Other:
- sheet Descret Input ports: added 24_OUT; removed GNDA
- sheet DiscretOut ports: added 24V_OUT; removed GND2
- moved on the sheet: C7

Commit message: all замменил резисторы failsafe в плате контроллера и обрал из перечня во всех остальных
Parts:
- R3, R6: now left out of the parts list
Changed lines of the file:
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@@
   )
   (symbol (lib_id "Device:R") (at 50.8 33.02 180) (unit 1)
-    (in_bom yes) (on_board yes) (dnp no)
+    (in_bom no) (on_board yes) (dnp no)
     (property "Reference" "R3" (at 45.72 33.02 90)
       (effects (font (size 1.27 1.27)))
@@
   )
   (symbol (lib_id "Device:R") (at 50.8 49.53 180) (unit 1)
-    (in_bom yes) (on_board yes) (dnp no)
+    (in_bom no) (on_board yes) (dnp no)
     (property "Reference" "R6" (at 48.26 50.8 90)
       (effects (font (size 1.27 1.27)))

Commit message: update schemas
Parts:
- F1: value 045201.5MRL -> 0451.5MRL (0.5 А)
- renumbered TP1 to G1, TP1 to GA1, TP1 to GD1, TP1 to TP62, TP1 to TP63, TP1 to TP64, TP1 to TP65, TP1 to TP66, TP1 to TP67, TP1 to TP68
