File: led_and_photodiode_board/led_and_photodiode_board.kicad_pcb (KiCad board)
At the start: 2 copper layers, 200 x 45 mm, 126 parts, among them J1 Conn_01x02_Socket, J2 DS1013-01-10RSiB-B, Q1 PT91-21B/TR7 (1206), Q2 PT91-21B/TR7 (1206), Q3 PT91-21B/TR7 (1206), Q4 PT91-21B/TR7 (1206), Q5 PT91-21B/TR7 (1206), Q6 PT91-21B/TR7 (1206), Q7 PT91-21B/TR7 (1206), Q8 PT91-21B/TR7 (1206)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

Commit message: led and photo топология
Parts:
- added C37: 0805 10nF 50V, Capacitor_SMD:C_0805_2012Metric, F.Cu at (188.5, 89.5)
- added C38: 0805 0,1uF 100V, Capacitor_SMD:C_0805_2012Metric, F.Cu at (61.9, 82.5)
- added C39: 0805 0,1uF 100V, Capacitor_SMD:C_0805_2012Metric, F.Cu at (146.9, 78.6)
- added D11: NUP2105L, Package_TO_SOT_SMD:SOT-23, F.Cu at (82.9, 86.4)
- added D12: NUP2105L, Package_TO_SOT_SMD:SOT-23, F.Cu at (118.0, 76.0)
- added D13: NUP2105L, Package_TO_SOT_SMD:SOT-23, F.Cu at (68.8, 87.0)
- added D14: NUP2105L, Package_TO_SOT_SMD:SOT-23, F.Cu at (139.7, 75.5)
- added R37: 1206 51 Ом, Resistor_SMD:R_1206_3216Metric, F.Cu at (191.8, 90.5)
- added R38: 2512 620 Ом, Resistor_SMD:R_2512_6332Metric, B.Cu at (75.5, 89.1)
- added R39: 2512 620 Ом, Resistor_SMD:R_2512_6332Metric, B.Cu at (121.6, 71.5)
- added R40: 2512 620 Ом, Resistor_SMD:R_2512_6332Metric, B.Cu at (79.4, 89.1)
- added R41: 2512 620 Ом, Resistor_SMD:R_2512_6332Metric, B.Cu at (125.5, 71.5)
- added R42: 2512 620 Ом, Resistor_SMD:R_2512_6332Metric, F.Cu at (64.8, 89.1)
- added R43: 2512 620 Ом, Resistor_SMD:R_2512_6332Metric, F.Cu at (60.8, 89.1)
- added R44: 2512 620 Ом, Resistor_SMD:R_2512_6332Metric, F.Cu at (147.8, 73.1)
- added R45: 2512 620 Ом, Resistor_SMD:R_2512_6332Metric, F.Cu at (143.9, 73.1)
- added U4: LM358, Package_SO:SOIC-8_3.9x4.9mm_P1.27mm, F.Cu at (67.3, 80.6)
- added U5: LM358, Package_SO:SOIC-8_3.9x4.9mm_P1.27mm, F.Cu at (141.2, 80.5)
- J1: footprint Connector:PAD_5x5_02 -> Connector_Wire:SolderWire-0.75sqmm_1x02_P7mm_D1.25mm_OD3.5mm
- R22, R25, R26, R28, R30, R32: moved to B.Cu
- U1, U2: value LM2901DR (SOIC-14) -> LM358; footprint Package_SO:SOIC-14_3.9x8.7mm_P1.27mm -> Package_SO:SOIC-8_3.9x4.9mm_P1.27mm
- U3: footprint Package_SO:HSOP-8-1EP_3.9x4.9mm_P1.27mm_EP2.3x2.3mm -> Package_SO:HSOP-8-1EP_3.9x4.9mm_P1.27mm_EP2.41x3.1mm
- moved G*** 112.6 mm to (197.6, 89.5)
- moved C35 64.9 mm to (77.0, 83.8), turned to 180 degrees
- moved C1 47.8 mm to (127.5, 85.0)
- moved TP14 18.3 mm to (130.1, 73.0)
- moved GA1 13.5 mm to (192.0, 78.4)
- moved R25 13.5 mm to (130.1, 76.0), turned to -90 degrees
- moved R31 13.1 mm to (147.8, 82.4)
- moved R28 12.6 mm to (129.3, 83.5), turned to 90 degrees
- moved TP15 12.5 mm to (134.5, 75.5)
- moved R27 12.2 mm to (130.7, 75.5)
- moved TP17 12.0 mm to (150.3, 80.8)
- moved R17 12.0 mm to (87.0, 80.8), turned to 180 degrees
- moved R32 10.8 mm to (143.5, 81.2), turned to 0 degrees
- moved R26 10.5 mm to (130.8, 83.5), turned to 90 degrees
- moved R20 10.2 mm to (62.1, 80.0), turned to 0 degrees
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Connections:
- C1 pad 1: /+24_FT_1 -> Net-(U2C-V+)
- C35 pad 1: /+24_FT_1 -> Net-(U1C-V+)
- R19 pad 2: Net-(U1C--) -> Net-(U4A--)
- R20 pad 2: Net-(U1D--) -> Net-(U4B--)
- R23 pad 2: Net-(U1C-+) -> Net-(U4A-+)
- R24 pad 2: Net-(U1D-+) -> Net-(U4B-+)
- R29 pad 2: Net-(U2C-+) -> Net-(U5A-+)
- R30 pad 2: Net-(U2C--) -> Net-(U5A--)
- R31 pad 2: Net-(U2D-+) -> Net-(U5B-+)
- R32 pad 2: Net-(U2D--) -> Net-(U5B--)
- U1 pad 1: /OUT4 -> /OUT3
- U1 pad 2: /OUT3 -> Net-(U1A--)
- U1 pad 3: /+24_FT_1 -> Net-(U1A-+)
- U1 pad 4: Net-(U1A--) -> GNDA
- U1 pad 5: Net-(U1A-+) -> Net-(U1B-+)
- U1 pad 7: Net-(U1B-+) -> /OUT4
- U1 pad 8: Net-(U1D--) -> Net-(U1C-V+)
- U2 pad 1: /OUT6 -> /OUT5
- U2 pad 2: /OUT5 -> Net-(U2A--)
- U2 pad 3: /+24_FT_1 -> Net-(U2A-+)
- U2 pad 4: Net-(U2A--) -> GNDA
- U2 pad 5: Net-(U2A-+) -> Net-(U2B-+)
- U2 pad 7: Net-(U2B-+) -> /OUT6
- U2 pad 8: Net-(U2D--) -> Net-(U2C-V+)
Routing:
- net /+24_FT_1: track 336.4 -> 371.0 mm
- net /OUT8: track 36.8 -> 55.9 mm
- net /Collector5: track 41.9 -> 25.5 mm, vias 3 -> 1
- net Net-(U2C-V+): track 0.00 -> 15.4 mm, vias 0 -> 1
- net /OUT2: track 59.2 -> 71.5 mm
- net /Collector8: track 84.2 -> 73.6 mm
- net GNDA: track 2.50 -> 13.0 mm, vias 253 -> 277
- net /OUT3: track 65.6 -> 55.6 mm
- net Net-(U4C-V+): track 0.00 -> 9.67 mm
- net /Collector3: track 39.1 -> 29.5 mm
- net Net-(U1C-V+): track 0.00 -> 9.47 mm, vias 0 -> 1
- net Net-(U5C-V+): track 0.00 -> 8.89 mm
- net /OUT6: track 38.9 -> 30.7 mm
- net Net-(U5A-+): track 0.00 -> 7.76 mm, vias 0 -> 1
- net Net-(U2C--): track 7.46 -> 0.00 mm
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Other:
- outline, holes or cut-outs redrawn

Commit message: refresh ledfotodiod
Parts:
- removed R37: 1206 51 Ом, Resistor_SMD:R_1206_3216Metric
- added R46: 2512 100 Ом, Resistor_SMD:R_2512_6332Metric_Pad1.40x3.35mm_HandSolder, B.Cu at (195.2, 86.3)
- added R47: 2512 100 Ом, Resistor_SMD:R_2512_6332Metric_Pad1.40x3.35mm_HandSolder, B.Cu at (195.2, 82.4)
- C37: moved to B.Cu
- D10: value 1N5819WS (SOD-323) -> B360; footprint Diode_SMD:D_SOD-323 -> Diode_SMD:D_SMC
- D9: value LL4148 (miniMELF) -> B360; footprint Diode_SMD:D_MiniMELF -> Diode_SMD:D_SMC
- R33: value opt (100k) -> 0805 160 кОм 5% - 0,125Вт
- moved G*** 31.0 mm to (167.6, 81.6)
- moved GA1 14.2 mm to (183.7, 89.9)
- moved C2 5.44 mm to (198.7, 78.3)
- moved C37 5.35 mm to (188.6, 84.2), turned to 180 degrees
- moved C10 4.13 mm to (199.3, 85.8), turned to 180 degrees
- moved C7 3.83 mm to (178.5, 76.0), turned to -90 degrees
- moved D9 3.83 mm to (189.3, 72.9)
- moved R35 3.14 mm to (177.6, 78.6)
- moved C36 2.37 mm to (199.3, 80.0), turned to 180 degrees
- moved L1 2.28 mm to (190.9, 81.9)
- moved D10 2.18 mm to (188.6, 88.9), turned to 0 degrees
- moved C9 2.10 mm to (174.7, 90.4)
- moved C8 1.90 mm to (180.7, 90.3)
- moved C6 1.71 mm to (187.2, 77.3)
- moved R34 1.10 mm to (180.5, 76.0), turned to -90 degrees
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Routing:
- net Net-(C37-Pad1): track 1.80 -> 8.44 mm
- net Net-(D10-K): track 22.5 -> 16.4 mm, vias 0 -> 3
- net Net-(D9-K): track 5.68 -> 7.29 mm
- net Net-(U3-FB): track 7.14 -> 5.76 mm
- net /Collector8: track 73.6 -> 74.7 mm
- net GNDA: vias 277 -> 293
- added copper zone on B.Cu, net Net-(D10-K)
- added copper zone on F.Cu, net Net-(D10-K)
- removed copper zone on B.Cu, net /+3.4V

Commit message: update schemas
Parts:
- moved G*** 11.3 mm to (177.9, 77.0)
Routing:
- net GNDA: vias 293 -> 289
Other:
- board text added: "PizzaBot inc."
- board text added: "t07v02a"
- board text removed: "t07 v02 a"
- board text removed: "{ "ViaStitching": "0.2", "stitch_zone_0": { "HSpacing": "1", "VSpacing": "1", "Clearance": "0", "Randomize": false } }"
