File: led_and_photodiode_board/led_and_photodiode_board.kicad_sch (KiCad schematic)
At the start: 46 parts, among them J1 Conn_01x02_Socket, J2 DS1013-01-10RSiB-B

Commit message: ledphoto обновлена схема и pcb
Parts:
- C11, C12, C13, C14, C15, C16, C17, C18, C2, C27, C28, C29, C3, C30, C31, C32, C33, C34: value 0,1uF 100V 0805 -> 0805 0,1uF 100V
- R1, R2, R3, R4, R5, R6, R7, R8: value 2512-100 Ом±5%-1 Вт -> 2512 68 Ом±5%-1 Вт
Connections:
- net +5V renamed +3.4V
Other:
- sheet DC-DC 24-5V ports: added +3,4V; removed +5V
Changed lines of the file:
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@@
 	)
 	(label "OUT3"
-		(at 143.51 74.93 0)
+		(at 143.51 69.85 0)
 		(fields_autoplaced yes)
 		(effects
@@
 	)
 	(label "Collector4"
-		(at 114.3 83.82 180)
+		(at 114.3 78.74 180)
 		(fields_autoplaced yes)
 		(effects
@@
 	)
 	(label "OUT4"
-		(at 143.51 77.47 0)
+		(at 143.51 72.39 0)
 		(fields_autoplaced yes)
 		(effects
@@
 	)
 	(label "OUT2"
-		(at 143.51 72.39 0)
+		(at 143.51 77.47 0)
 		(fields_autoplaced yes)
 		(effects
@@
 	)
 	(label "Collector2"
-		(at 114.3 78.74 180)
+		(at 114.3 83.82 180)
 		(fields_autoplaced yes)
 		(effects
@@
 	)
 	(label "Collector3"
-		(at 114.3 81.28 180)
+		(at 114.3 76.2 180)
 		(fields_autoplaced yes)
 		(effects
@@
 	)
 	(label "OUT1"
-		(at 143.51 69.85 0)
+		(at 143.51 74.93 0)
 		(fields_autoplaced yes)
 		(effects
@@
 		)
 	)
-	(label "Collector3"
-		(at 72.39 92.71 0)
+	(label "+3.4V"
+		(at 38.1 27.94 180)
 		(fields_autoplaced yes)
 		(effects
@@
 				(size 1.27 1.27)
 			)
-			(justify left bottom)
+			(justify right bottom)
 		)
 	)
-	(label "+5V"
-		(at 38.1 27.94 180)
+	(label "Collector3"
+		(at 72.39 92.71 0)
 		(fields_autoplaced yes)
 		(effects
@@
 				(size 1.27 1.27)
 			)
-			(justify right bottom)
+			(justify left bottom)
 		)
 	)
@@
 		)
 	)
-	(label "+5V"
+	(label "+3.4V"
 		(at 251.46 80.01 0)
 		(fields_autoplaced yes)
@@
 	)
 	(label "Collector1"
-		(at 114.3 76.2 180)
+		(at 114.3 81.28 180)
 		(fields_autoplaced yes)
 		(effects
@@
 			)
 		)
-		(property "Value" "0,1uF 100V 0805"
+		(property "Value" "0805 0,1uF 100V"
 			(at 261.62 57.15 90)
 			(effects
@@
 			)
 		)
-		(property "Value" "2512-100 Ом±5%-1 Вт"
+		(property "Value" "2512 68 Ом±5%-1 Вт"
 			(at 241.3 34.29 0)
 			(effects
@@
 			)
 		)
-		(property "Value" "0,1uF 100V 0805"
+		(property "Value" "0805 0,1uF 100V"
 			(at 205.74 57.15 90)
 			(effects
@@
 			)
 		)
-		(property "Value" "0,1uF 100V 0805"
+		(property "Value" "0805 0,1uF 100V"
 			(at 259.08 124.46 90)
 			(effects
@@
 			)
 		)
-		(property "Value" "2512-100 Ом±5%-1 Вт"
+		(property "Value" "2512 68 Ом±5%-1 Вт"
 			(at 211.582 57.404 0)
 			(effects
@@
 			)
 		)
-		(property "Value" "2512-100 Ом±5%-1 Вт"
+		(property "Value" "2512 68 Ом±5%-1 Вт"
 			(at 110.236 58.42 0)
 			(effects
@@
 			)
 		)
-		(property "Value" "0,1uF 100V 0805"
+		(property "Value" "0805 0,1uF 100V"
 			(at 107.95 57.15 90)
 			(effects
@@
 			)
 		)
-		(property "Value" "2512-100 Ом±5%-1 Вт"
+		(property "Value" "2512 68 Ом±5%-1 Вт"
 			(at 138.43 34.29 0)
 			(effects
@@
 			)
 		)
-		(property "Value" "0,1uF 100V 0805"
+		(property "Value" "0805 0,1uF 100V"
 			(at 176.53 124.46 90)
 			(effects
@@
 			)
 		)
-		(property "Value" "2512-100 Ом±5%-1 Вт"
+		(property "Value" "2512 68 Ом±5%-1 Вт"
 			(at 57.404 57.912 0)
 			(effects
@@
 			)
 		)
-		(property "Value" "0,1uF 100V 0805"
+		(property "Value" "0805 0,1uF 100V"
 			(at 153.67 124.46 90)
 			(effects
@@
 			)
 		)
-		(property "Value" "2512-100 Ом±5%-1 Вт"
+		(property "Value" "2512 68 Ом±5%-1 Вт"
 			(at 187.96 34.29 0)
 			(effects
@@
 			)
 		)
-		(property "Value" "2512-100 Ом±5%-1 Вт"
+		(property "Value" "2512 68 Ом±5%-1 Вт"
 			(at 90.17 34.29 0)
 			(effects
@@
 			)
 		)
-		(property "Value" "0,1uF 100V 0805"
+		(property "Value" "0805 0,1uF 100V"
 			(at 248.92 124.46 90)
 			(effects
@@
 			)
 		)
-		(property "Value" "0,1uF 100V 0805"
+		(property "Value" "0805 0,1uF 100V"
 			(at 157.48 57.15 90)
 			(effects
@@
 			)
 		)
-		(property "Value" "0,1uF 100V 0805"
+		(property "Value" "0805 0,1uF 100V"
 			(at 233.68 38.1 90)
 			(effects
@@
 			)
 		)
-		(property "Value" "0,1uF 100V 0805"
+		(property "Value" "0805 0,1uF 100V"
 			(at 132.08 38.1 90)
 			(effects
@@
 			)
 		)
-		(property "Value" "0,1uF 100V 0805"
+		(property "Value" "0805 0,1uF 100V"
 			(at 226.06 124.46 90)
 			(effects
@@
 			)
 		)
-		(property "Value" "0,1uF 100V 0805"
+		(property "Value" "0805 0,1uF 100V"
 			(at 186.69 124.46 90)
 			(effects
@@
 			)
 		)
-		(property "Value" "0,1uF 100V 0805"
+		(property "Value" "0805 0,1uF 100V"
 			(at 83.82 38.1 90)
 			(effects
@@
 			)
 		)
-		(property "Value" "0,1uF 100V 0805"
+		(property "Value" "0805 0,1uF 100V"
 			(at 237.49 124.46 90)
 			(effects
@@
 			)
 		)
-		(property "Value" "0,1uF 100V 0805"
+		(property "Value" "0805 0,1uF 100V"
 			(at 45.72 46.99 0)
 			(effects
@@
 			)
 		)
-		(property "Value" "0,1uF 100V 0805"
+		(property "Value" "0805 0,1uF 100V"
 			(at 165.1 124.46 90)
 			(effects
@@
 			)
 		)
-		(property "Value" "0,1uF 100V 0805"
+		(property "Value" "0805 0,1uF 100V"
 			(at 48.26 90.17 90)
 			(effects
@@
 			)
 		)
-		(property "Value" "0,1uF 100V 0805"
+		(property "Value" "0805 0,1uF 100V"
 			(at 181.61 38.1 90)
 			(effects
@@
 			)
 		)
-		(property "Value" "2512-100 Ом±5%-1 Вт"
+		(property "Value" "2512 68 Ом±5%-1 Вт"
 			(at 160.782 57.658 0)
 			(effects
@@
 			)
 		)
-		(pin "+5V" output
-			(at 251.46 80.01 0)
+		(pin "+24V" input
+			(at 227.33 80.01 180)
 			(effects
 				(font
 					(size 1.27 1.27)
 				)
-				(justify right)
+				(justify left)
 			)
 		)
-		(pin "+24V" input
-			(at 227.33 80.01 180)
+		(pin "+3,4V" output
+			(at 251.46 80.01 0)
 			(effects
 				(font
 					(size 1.27 1.27)
 				)
-				(justify left)
+				(justify right)
 			)
 		)

Commit message: led and photo топология
Parts:
- J1: footprint Connector:PAD_5x5_02 -> Connector_Wire:SolderWire-0.75sqmm_1x02_P7mm_D1.25mm_OD3.5mm
Changed lines of the file:
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@@
 			)
 		)
-		(property "Footprint" "Connector:PAD_5x5_02"
+		(property "Footprint" "Connector_Wire:SolderWire-0.75sqmm_1x02_P7mm_D1.25mm_OD3.5mm"
 			(at 115.57 168.91 0)
 			(effects

Commit message: update schemas
Parts:
- GA1, TP1, TP2, TP3, TP4, TP5, TP6, TP7, TP8, TP9: now left out of the parts list
Changed lines of the file:
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@@
 		(unit 1)
 		(exclude_from_sim no)
-		(in_bom yes)
+		(in_bom no)
 		(on_board yes)
 		(dnp no)
@@
 		(unit 1)
 		(exclude_from_sim no)
-		(in_bom yes)
+		(in_bom no)
 		(on_board yes)
 		(dnp no)
@@
 		(unit 1)
 		(exclude_from_sim no)
-		(in_bom yes)
+		(in_bom no)
 		(on_board yes)
 		(dnp no)
@@
 		(unit 1)
 		(exclude_from_sim no)
-		(in_bom yes)
+		(in_bom no)
 		(on_board yes)
 		(dnp no)
@@
 		(unit 1)
 		(exclude_from_sim no)
-		(in_bom yes)
+		(in_bom no)
 		(on_board yes)
 		(dnp no)
@@
 		(unit 1)
 		(exclude_from_sim no)
-		(in_bom yes)
+		(in_bom no)
 		(on_board yes)
 		(dnp no)
@@
 		(unit 1)
 		(exclude_from_sim no)
-		(in_bom yes)
+		(in_bom no)
 		(on_board yes)
 		(dnp no)
@@
 		(unit 1)
 		(exclude_from_sim no)
-		(in_bom yes)
+		(in_bom no)
 		(on_board yes)
 		(dnp no)
@@
 		(unit 1)
 		(exclude_from_sim no)
-		(in_bom yes)
+		(in_bom no)
 		(on_board yes)
 		(dnp no)
@@
 		(unit 1)
 		(exclude_from_sim no)
-		(in_bom yes)
+		(in_bom no)
 		(on_board yes)
 		(dnp no)
