File: step_motor_board/Stepper_Motor_Control.kicad_sch (KiCad schematic)
At the start: 57 parts, among them J2 Driver (DG141R-10), Q1 2SC2712 (SOT-23), Q2 2SC2712 (SOT-23), Q3 2SC2712 (SOT-23), U4 PAI141M30 (SOIC-16), U6 L78L05 (SOT89-3), U8 74LVC2G14 (SOT-23-6)

Commit message: DC, contr, mb, step v2
Parts:
- C15, C16, C17, C19, C20, C21, C24, C40, C41: value 0,1uF 50V 0603 -> 0,1uF 100V 0603
- C9: renamed from C39; value 0,1uF 100V 0805 -> 0,1uF 100V 0603; footprint PCM_Capacitor_SMD_AKL:C_0805_2012Metric_Pad1.18x1.45mm_HandSolder -> Capacitor_SMD:C_0603_1608Metric_Pad1.08x0.95mm_HandSolder
- C9: renamed from C18; value 0,1uF 100V 0805 -> 0,1uF 100V 0603; footprint PCM_Capacitor_SMD_AKL:C_0805_2012Metric_Pad1.18x1.45mm_HandSolder -> Capacitor_SMD:C_0603_1608Metric_Pad1.08x0.95mm_HandSolder
- J2: value Driver (DG141R-10) -> DG141R-2.54-10P-14-00A(H) (Driver)
- R12: renamed from R15; value 0805-10 кОм±5%-0,125 Вт -> 0603-10 кОм±5%-0,0625 Вт; footprint PCM_4ms_Resistor:R_0805_2012Metric -> Resistor_SMD:R_0603_1608Metric
- R13: renamed from R16; value 0805-10 кОм±5%-0,125 Вт -> 0603-10 кОм±5%-0,0625 Вт; footprint PCM_4ms_Resistor:R_0805_2012Metric -> Resistor_SMD:R_0603_1608Metric
- R14: renamed from R17; value 0805-10 кОм±5%-0,125 Вт -> 0603-10 кОм±5%-0,0625 Вт; footprint PCM_4ms_Resistor:R_0805_2012Metric -> Resistor_SMD:R_0603_1608Metric
- R16: renamed from R46; value 0805-1 кОм±5%-0,125 Вт -> 0603-1 кОм±5%-0,0625 Вт; footprint PCM_Resistor_SMD_AKL:R_0805_2012Metric_Pad1.20x1.40mm_HandSolder -> Resistor_SMD:R_0603_1608Metric
- R16: renamed from R43; value 0805-1 кОм±5%-0,125 Вт -> 0603-1 кОм±5%-0,0625 Вт; footprint PCM_Resistor_SMD_AKL:R_0805_2012Metric_Pad1.20x1.40mm_HandSolder -> Resistor_SMD:R_0603_1608Metric
- R25: renamed from R45; value 0805-10 кОм±5%-0,125 Вт -> 0603-10 кОм±5%-0,0625 Вт; footprint PCM_Resistor_SMD_AKL:R_0805_2012Metric_Pad1.20x1.40mm_HandSolder -> Resistor_SMD:R_0603_1608Metric
- R25: renamed from R44; value 0805-10 кОм±5%-0,125 Вт -> 0603-10 кОм±5%-0,0625 Вт; footprint PCM_Resistor_SMD_AKL:R_0805_2012Metric_Pad1.20x1.40mm_HandSolder -> Resistor_SMD:R_0603_1608Metric
- R26: renamed from R13; value 0603-10 кОм±5%-0,062 Вт -> 0603-1.5 кОм±5%-0,062 Вт; footprint PCM_Resistor_SMD_AKL:R_0603_1608Metric_Pad1.05x0.95mm_HandSolder -> Resistor_SMD:R_0603_1608Metric
- R26: renamed from R42; footprint PCM_Resistor_SMD_AKL:R_1206_3216Metric_Pad1.42x1.75mm_HandSolder -> Resistor_SMD:R_1206_3216Metric
- R26: renamed from R41; footprint PCM_Resistor_SMD_AKL:R_1206_3216Metric_Pad1.42x1.75mm_HandSolder -> Resistor_SMD:R_1206_3216Metric
- R26: renamed from R21; value 0603-10 кОм±5%-0,062 Вт -> 0603-1.5 кОм±5%-0,062 Вт; footprint PCM_Resistor_SMD_AKL:R_0603_1608Metric_Pad1.05x0.95mm_HandSolder -> Resistor_SMD:R_0603_1608Metric
- R26: renamed from R39; footprint PCM_Resistor_SMD_AKL:R_1206_3216Metric_Pad1.42x1.75mm_HandSolder -> Resistor_SMD:R_1206_3216Metric
- R26: renamed from R9; value 2512-2,4 кОм±5%-1 Вт -> 2512-1,3 кОм±5%-1 Вт
- R26: renamed from R14; value 0603-10 кОм±5%-0,062 Вт -> 0603-270 Ом±5%-0,062 Вт; footprint PCM_Resistor_SMD_AKL:R_0603_1608Metric_Pad1.05x0.95mm_HandSolder -> Resistor_SMD:R_0603_1608Metric
- R26: renamed from R20; value 2512-2,4 кОм±5%-1 Вт -> 2512-1,3 кОм±5%-1 Вт
- R26: renamed from R10; value 0603-10 кОм±5%-0,062 Вт -> 0603-1.5 кОм±5%-0,062 Вт; footprint PCM_Resistor_SMD_AKL:R_0603_1608Metric_Pad1.05x0.95mm_HandSolder -> Resistor_SMD:R_0603_1608Metric
- R26: renamed from R12; value 2512-2,4 кОм±5%-1 Вт -> 2512-1,3 кОм±5%-1 Вт
- R26: renamed from R22; value 0603-10 кОм±5%-0,062 Вт -> 0603-270 Ом±5%-0,062 Вт; footprint PCM_Resistor_SMD_AKL:R_0603_1608Metric_Pad1.05x0.95mm_HandSolder -> Resistor_SMD:R_0603_1608Metric
- R26: renamed from R11; value 0603-10 кОм±5%-0,062 Вт -> 0603-270 Ом±5%-0,062 Вт; footprint PCM_Resistor_SMD_AKL:R_0603_1608Metric_Pad1.05x0.95mm_HandSolder -> Resistor_SMD:R_0603_1608Metric
- R26: renamed from R40; footprint PCM_Resistor_SMD_AKL:R_1206_3216Metric_Pad1.42x1.75mm_HandSolder -> Resistor_SMD:R_1206_3216Metric
- U4: value PAI141M30 (SOIC-16) -> Pai141M30 (SOIC-16)
- renumbered R47 to R26, R19 to R4, R18 to R4
Other:
- moved on the sheet: C37, C38, R12, R13, R14, R25, TP18, TP19

Commit message: all замменил резисторы failsafe в плате контроллера и обрал из перечня во всех остальных
Parts:
- C15, C16, C17, C19, C20, C21, C23, C24, C40, C41: footprint Capacitor_SMD:C_0603_1608Metric_Pad1.08x0.95mm_HandSolder -> Capacitor_SMD:C_0603_1608Metric
- C18, C39: renamed from C9; footprint Capacitor_SMD:C_0603_1608Metric_Pad1.08x0.95mm_HandSolder -> Capacitor_SMD:C_0603_1608Metric
- C37, C38: footprint PCM_Capacitor_SMD_US_Handsoldering_AKL:C_0603_1608Metric_Pad1.08x0.95mm -> Capacitor_SMD:C_0603_1608Metric
- J2: value DG141R-2.54-10P-14-00A(H) (Driver) -> DG141R-2.54-10P-14-00A(H) (Driver)
- Q1, Q2, Q3: footprint PCM_Package_TO_SOT_SMD_AKL:SOT-23 -> Package_TO_SOT_SMD:SOT-23
- R12, R20, R9: renamed from R26; footprint PCM_Resistor_SMD_AKL:R_2512_6332Metric_Pad1.52x3.35mm_HandSolder -> Resistor_SMD:R_2512_6332Metric
- R18, R19: renamed from R4; footprint PCM_4ms_Resistor:R_0805_2012Metric -> Resistor_SMD:R_0805_2012Metric
- R47: renamed from R26; footprint PCM_Resistor_SMD_AKL:R_1206_3216Metric_Pad1.42x1.75mm_HandSolder -> Resistor_SMD:R_1206_3216Metric
- TP10, TP18, TP19, TP20, TP21, TP22, TP23, TP3, TP8, TP9: footprint PCM_4ms_TestPoint:TestPoint_D1 -> TestPoint:TestPoint_Pad_D1.0mm
- renumbered R26 to R10, R26 to R11, R26 to R13, R26 to R14, R12 to R15, R13 to R16, R14 to R17, R26 to R21, R26 to R22, R26 to R39, R26 to R40, R26 to R41, R26 to R42, R16 to R43, R25 to R44, R25 to R45, R16 to R46

Commit message: update schemas
Changed lines of the file:
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@@
 (kicad_sch
-	(version 20231120)
+	(version 20250114)
 	(generator "eeschema")
-	(generator_version "8.0")
+	(generator_version "9.0")
 	(paper "A4")
 	(junction
@@
 	(label "EN_out-"
 		(at 30.48 41.91 0)
-		(fields_autoplaced yes)
 		(effects
 			(font
@@
 	(label "IN_POSITION"
 		(at 232.41 133.35 0)
-		(fields_autoplaced yes)
 		(effects
 			(font
@@
 	(label "IN_POSITION_out+"
 		(at 85.09 54.61 0)
-		(fields_autoplaced yes)
 		(effects
 			(font
@@
 	(label "DIR"
 		(at 254 50.8 0)
-		(fields_autoplaced yes)
 		(effects
 			(font
@@
 	(label "ALARM_out+"
 		(at 57.15 124.46 180)
-		(fields_autoplaced yes)
 		(effects
 			(font
@@
 	(label "ALARM_out+"
 		(at 88.9 59.69 0)
-		(fields_autoplaced yes)
 		(effects
 			(font
@@
 	(label "EN_out-"
 		(at 113.03 22.86 180)
-		(fields_autoplaced yes)
 		(effects
 			(font
@@
 	(label "DIR_out-"
 		(at 111.76 45.72 180)
-		(fields_autoplaced yes)
 		(effects
 			(font
@@
 	(label "STEP_out-"
 		(at 113.03 64.77 180)
-		(fields_autoplaced yes)
 		(effects
 			(font
@@
 	(label "EN"
 		(at 254 48.26 0)
-		(fields_autoplaced yes)
 		(effects
 			(font
@@
 	(label "IN_POSITION_out+"
 		(at 57.15 135.89 180)
-		(fields_autoplaced yes)
 		(effects
 			(font
@@
 	(label "DIR_out-"
 		(at 30.48 46.99 0)
-		(fields_autoplaced yes)
 		(effects
 			(font
@@
 	(label "STEP_out-"
 		(at 30.48 52.07 0)
-		(fields_autoplaced yes)
 		(effects
 			(font
@@
 	(label "STEP"
 		(at 254 53.34 0)
-		(fields_autoplaced yes)
 		(effects
 			(font
@@
 	(label "ALARM"
 		(at 232.41 110.49 0)
-		(fields_autoplaced yes)
 		(effects
 			(font
@@
 		(shape input)
 		(at 264.16 48.26 0)
-		(fields_autoplaced yes)
 		(effects
 			(font
@@
 		(shape input)
 		(at 255.27 133.35 0)
-		(fields_autoplaced yes)
 		(effects
 			(font
@@
 		(shape input)
 		(at 264.16 50.8 0)
-		(fields_autoplaced yes)
 		(effects
 			(font
@@
 		(shape input)
 		(at 264.16 53.34 0)
-		(fields_autoplaced yes)
 		(effects
 			(font
@@
 		(shape input)
 		(at 255.27 110.49 0)
-		(fields_autoplaced yes)
-		(effects
-			(font
+		(effects
+			(font
