File: triac_board/Simister.kicad_sch (KiCad schematic)
At the start: 12 parts, among them Q1 DTC114ECA (SOT-23), Q3 BTA41-600B (TO-218)

Commit message: Triak v2.1
Parts:
- C23: value 0,1uF 50V 0805 -> 0,1uF 100V 0603; footprint Capacitor_SMD:C_0805_2012Metric_Pad1.18x1.45mm_HandSolder -> Capacitor_SMD:C_0603_1608Metric
Changed lines of the file:
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@@
   )
   (symbol (lib_id "Device:R") (at 114.3 52.07 270) (unit 1)
-    (in_bom yes) (on_board yes) (dnp no) (fields_autoplaced)
+    (in_bom yes) (on_board yes) (dnp no)
     (property "Reference" "R12" (at 114.3 45.72 90)
       (effects (font (size 1.27 1.27)))
     )
-    (property "Value" "2512-180 Ом±5%-1 Вт" (at 114.3 48.26 90)
+    (property "Value" "2512-180 Ом±5%-1 Вт" (at 113.03 55.88 90)
       (effects (font (size 1.27 1.27)))
     )
@@
     (pin "1")
     (instances
-      (project "Плата симистров"
+      (project "triac_board"
         (path "/271a56a4-fac2-444b-8acf-7cf36bf0ab17/997d7511-5408-445d-86dd-063aa13180e2/a92943f3-fb5f-4928-a4c6-18ad14104b9b"
           (reference "R12") (unit 1)
@@
     (pin "1")
     (instances
-      (project "Плата симистров"
+      (project "triac_board"
         (path "/271a56a4-fac2-444b-8acf-7cf36bf0ab17/997d7511-5408-445d-86dd-063aa13180e2"
           (reference "#PWR049") (unit 1)
@@
     (pin "1")
     (instances
-      (project "Плата симистров"
+      (project "triac_board"
         (path "/271a56a4-fac2-444b-8acf-7cf36bf0ab17/997d7511-5408-445d-86dd-063aa13180e2/63b095b4-3c9c-489d-b37a-8fc245f2b355"
           (reference "C28") (unit 1)
@@
     (pin "1")
     (instances
-      (project "Плата симистров"
+      (project "triac_board"
         (path "/271a56a4-fac2-444b-8acf-7cf36bf0ab17/997d7511-5408-445d-86dd-063aa13180e2/a92943f3-fb5f-4928-a4c6-18ad14104b9b"
           (reference "C18") (unit 1)
@@
     (pin "1")
     (instances
-      (project "Плата симистров"
+      (project "triac_board"
         (path "/271a56a4-fac2-444b-8acf-7cf36bf0ab17/997d7511-5408-445d-86dd-063aa13180e2/a92943f3-fb5f-4928-a4c6-18ad14104b9b"
           (reference "TP11") (unit 1)
@@
       (effects (font (size 1.27 1.27)) (justify left))
     )
-    (property "Value" "0,1uF 50V 0805" (at 73.66 54.61 0)
-      (effects (font (size 1.27 1.27)) (justify left))
-    )
-    (property "Footprint" "Capacitor_SMD:C_0805_2012Metric_Pad1.18x1.45mm_HandSolder" (at 76.5048 52.07 0)
+    (property "Value" "0,1uF 100V 0603" (at 73.66 54.61 0)
+      (effects (font (size 1.27 1.27)) (justify left))
+    )
+    (property "Footprint" "Capacitor_SMD:C_0603_1608Metric" (at 76.5048 52.07 0)
       (effects (font (size 1.27 1.27)) hide)
     )
@@
     (pin "1")
     (instances
-      (project "Плата симистров"
+      (project "triac_board"
         (path "/271a56a4-fac2-444b-8acf-7cf36bf0ab17/997d7511-5408-445d-86dd-063aa13180e2"
           (reference "C23") (unit 1)
@@
     (pin "1")
     (instances
-      (project "Плата симистров"
+      (project "triac_board"
         (path "/271a56a4-fac2-444b-8acf-7cf36bf0ab17/997d7511-5408-445d-86dd-063aa13180e2/a92943f3-fb5f-4928-a4c6-18ad14104b9b"
           (reference "R13") (unit 1)
@@
     (pin "2")
     (instances
-      (project "Плата симистров"
+      (project "triac_board"
         (path "/271a56a4-fac2-444b-8acf-7cf36bf0ab17"
           (reference "Q1") (unit 1)
@@
     (pin "1")
     (instances
-      (project "Плата симистров"
+      (project "triac_board"
         (path "/271a56a4-fac2-444b-8acf-7cf36bf0ab17/997d7511-5408-445d-86dd-063aa13180e2/a92943f3-fb5f-4928-a4c6-18ad14104b9b"
           (reference "Q3") (unit 1)
@@
     (pin "3")
     (instances
-      (project "Плата симистров"
+      (project "triac_board"
         (path "/271a56a4-fac2-444b-8acf-7cf36bf0ab17/997d7511-5408-445d-86dd-063aa13180e2/63b095b4-3c9c-489d-b37a-8fc245f2b355"
           (reference "OC5") (unit 1)
@@
     (pin "1")
     (instances
-      (project "Плата симистров"
+      (project "triac_board"
         (path "/271a56a4-fac2-444b-8acf-7cf36bf0ab17/997d7511-5408-445d-86dd-063aa13180e2/a92943f3-fb5f-4928-a4c6-18ad14104b9b"
           (reference "R14") (unit 1)
@@
     (pin "1")
     (instances
-      (project "Плата симистров"
+      (project "triac_board"
         (path "/271a56a4-fac2-444b-8acf-7cf36bf0ab17/997d7511-5408-445d-86dd-063aa13180e2/a92943f3-fb5f-4928-a4c6-18ad14104b9b"
           (reference "R15") (unit 1)
@@
     (pin "1")
     (instances
-      (project "Плата симистров"
+      (project "triac_board"
         (path "/271a56a4-fac2-444b-8acf-7cf36bf0ab17/997d7511-5408-445d-86dd-063aa13180e2/a92943f3-fb5f-4928-a4c6-18ad14104b9b"
           (reference "TP12") (unit 1)
@@
     (pin "1")
     (instances
-      (project "Плата симистров"
+      (project "triac_board"
         (path "/271a56a4-fac2-444b-8acf-7cf36bf0ab17"
           (reference "#PWR021") (unit 1)

Commit message: triak обновлен снаббер
Parts:
- R14: value 2512-51 Ом±5%-1 Вт -> 2512-2 кОм±5%-1 Вт
Changed lines of the file:
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@@
       (effects (font (size 1.27 1.27)) (justify right))
     )
-    (property "Value" "2512-51 Ом±5%-1 Вт" (at 167.64 62.23 0)
+    (property "Value" "2512-2 кОм±5%-1 Вт" (at 167.64 62.23 0)
       (effects (font (size 1.27 1.27)) (justify right))
     )

Commit message: triak убраны тестовые площадки с 220в
Parts:
- removed TP12: TestPoint, PCM_4ms_TestPoint:TestPoint_D1, symbol Connector:TestPoint
- R12, R13, R14: footprint PCM_Resistor_SMD_AKL:R_2512_6332Metric -> Resistor_SMD:R_2512_6332Metric
Changed lines of the file:
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@@
   (junction (at 133.35 52.07) (diameter 0) (color 0 0 0 0)
   )
-  (junction (at 179.07 85.09) (diameter 0) (color 0 0 0 0)
-  )
   (junction (at 119.38 52.07) (diameter 0) (color 0 0 0 0)
   )
@@
     (stroke (width 0) (type default))
   )
-  (wire (pts (xy 179.07 85.09) (xy 196.85 85.09))
-    (stroke (width 0) (type default))
-  )
   (wire (pts (xy 77.47 62.23) (xy 66.04 62.23))
     (stroke (width 0) (type default))
@@
     (stroke (width 0) (type default))
   )
-  (wire (pts (xy 165.1 85.09) (xy 179.07 85.09))
+  (wire (pts (xy 165.1 85.09) (xy 196.85 85.09))
     (stroke (width 0) (type default))
   )
@@
       (effects (font (size 1.27 1.27)))
     )
-    (property "Footprint" "PCM_Resistor_SMD_AKL:R_2512_6332Metric" (at 114.3 50.292 90)
+    (property "Footprint" "Resistor_SMD:R_2512_6332Metric" (at 114.3 50.292 90)
       (effects (font (size 1.27 1.27)) hide)
     )
@@
       (effects (font (size 1.27 1.27)))
     )
-    (property "Footprint" "PCM_Resistor_SMD_AKL:R_2512_6332Metric" (at 125.73 50.292 90)
+    (property "Footprint" "Resistor_SMD:R_2512_6332Metric" (at 125.73 50.292 90)
       (effects (font (size 1.27 1.27)) hide)
     )
@@
       (effects (font (size 1.27 1.27)) (justify right))
     )
-    (property "Footprint" "PCM_Resistor_SMD_AKL:R_2512_6332Metric" (at 166.878 60.96 90)
+    (property "Footprint" "Resistor_SMD:R_2512_6332Metric" (at 166.878 60.96 90)
       (effects (font (size 1.27 1.27)) hide)
     )
@@
         )
       )
-    )
-  )
-  (symbol (lib_id "Connector:TestPoint") (at 179.07 85.09 0) (unit 1)
-    (in_bom no) (on_board yes) (dnp no) (fields_autoplaced)
-    (property "Reference" "TP12" (at 181.61 80.518 0)
-      (effects (font (size 1.27 1.27)) (justify left))
-    )
-    (property "Value" "TestPoint" (at 181.61 83.058 0)
-      (effects (font (size 1.27 1.27)) (justify left) hide)
-    )
-    (property "Footprint" "PCM_4ms_TestPoint:TestPoint_D1" (at 184.15 85.09 0)
-      (effects (font (size 1.27 1.27)) hide)
-    )
-    (property "Datasheet" "~" (at 184.15 85.09 0)
-      (effects (font (size 1.27 1.27)) hide)
-    )
-    (pin "1")
-    (instances
-      (project "triac_board"
-        (path "/271a56a4-fac2-444b-8acf-7cf36bf0ab17/997d7511-5408-445d-86dd-063aa13180e2/a92943f3-fb5f-4928-a4c6-18ad14104b9b"
-          (reference "TP12") (unit 1)
-        )
-        (path "/271a56a4-fac2-444b-8acf-7cf36bf0ab17/997d7511-5408-445d-86dd-063aa13180e2/dcab90d0-6412-4eeb-8218-0c0b15cdd6ab"
-          (reference "TP14") (unit 1)
-        )
-        (path "/271a56a4-fac2-444b-8acf-7cf36bf0ab17/997d7511-5408-445d-86dd-063aa13180e2/f2cea334-e45e-49d8-bc5b-499bf5169a47"
-          (reference "TP16") (unit 1)
-        )
-        (path "/271a56a4-fac2-444b-8acf-7cf36bf0ab17/997d7511-5408-445d-86dd-063aa13180e2/63b095b4-3c9c-489d-b37a-8fc245f2b355"
-          (reference "TP18") (unit 1)
-        )
-      )
-      (project "Плата внешних шаговых двигателей"
-        (path "/7f8f7dc9-8c50-44ed-985c-35a6d8c67be0/0d239b34-7914-40bc-9b83-7e562c30defe"
-          (reference "TP21") (unit 1)
-        )
-        (path "/7f8f7dc9-8c50-44ed-985c-35a6d8c67be0/1f6eaeee-a46e-4730-b225-3a410300814a"
-          (reference "TP5") (unit 1)
-        )
-      )

Commit message: triak снаббер
Parts:
- removed C28: 0,01uF 600V 1206 (GRM31BR72J103KW01L), Capacitor_SMD:C_1206_3216Metric_Pad1.33x1.80mm_HandSolder, symbol Device:C
- added C19: 0,01uF 630V (CL11-103K/630V), Capacitor_THT:C_Rect_L7.0mm_W4.5mm_P5.00mm, symbol Device:C
- C18: value 0,01uF 600V 1206 (GRM31BR72J103KW01L) -> 0,01uF 630V (CL11-103K/630V); footprint Capacitor_SMD:C_1206_3216Metric_Pad1.33x1.80mm_HandSolder -> Capacitor_THT:C_Rect_L7.0mm_W4.5mm_P5.00mm
- R12: value 2512-180 Ом±5%-1 Вт -> 0207 MELF -180 Ом±5%-1 Вт; footprint Resistor_SMD:R_2512_6332Metric -> Resistor_SMD:R_MELF_MMB-0207
- R13: value 2512-1 кОм±5%-1 Вт -> 0207 MELF -1 кОм±5%-1 Вт; footprint Resistor_SMD:R_2512_6332Metric -> Resistor_SMD:R_MELF_MMB-0207
- R14: value 2512-2 кОм±5%-1 Вт -> 0207 MELF -2 кОм±5%-1 Вт; footprint Resistor_SMD:R_2512_6332Metric -> Resistor_SMD:R_MELF_MMB-0207
Connections:
- net AC_OUT: now also C19.2
- net at R12.1, R13.2: now also C19.1
Changed lines of the file:
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@@
       (effects (font (size 1.27 1.27)))
     )
-    (property "Value" "2512-180 Ом±5%-1 Вт" (at 113.03 55.88 90)
-      (effects (font (size 1.27 1.27)))
-    )
-    (property "Footprint" "Resistor_SMD:R_2512_6332Metric" (at 114.3 50.292 90)
+    (property "Value" "0207 MELF -180 Ом±5%-1 Вт" (at 113.03 55.88 90)
+      (effects (font (size 1.27 1.27)))
+    )
+    (property "Footprint" "Resistor_SMD:R_MELF_MMB-0207" (at 114.3 50.292 90)
       (effects (font (size 1.27 1.27)) hide)
     )
@@
     )
   )
-  (symbol (lib_id "Device:C") (at 119.38 80.01 0) (unit 1)
-    (in_bom yes) (on_board yes) (dnp no)
-    (property "Reference" "C28" (at 114.3 83.82 0)
-      (effects (font (size 1.27 1.27)) (justify left))
-    )
-    (property "Value" "0,01uF 600V 1206 (GRM31BR72J103KW01L)" (at 109.22 87.63 0)
-      (effects (font (size 1.27 1.27)) (justify left))
-    )
-    (property "Footprint" "Capacitor_SMD:C_1206_3216Metric_Pad1.33x1.80mm_HandSolder" (at 120.3452 83.82 0)
-      (effects (font (size 1.27 1.27)) hide)
-    )
-    (property "Datasheet" "~" (at 119.38 80.01 0)
-      (effects (font (size 1.27 1.27)) hide)
-    )
-    (pin "2")
-    (pin "1")
-    (instances
-      (project "triac_board"
-        (path "/271a56a4-fac2-444b-8acf-7cf36bf0ab17/997d7511-5408-445d-86dd-063aa13180e2/63b095b4-3c9c-489d-b37a-8fc245f2b355"
-          (reference "C28") (unit 1)
-        )
-        (path "/271a56a4-fac2-444b-8acf-7cf36bf0ab17/997d7511-5408-445d-86dd-063aa13180e2/a92943f3-fb5f-4928-a4c6-18ad14104b9b"
-          (reference "C19") (unit 1)
-        )
-        (path "/271a56a4-fac2-444b-8acf-7cf36bf0ab17/997d7511-5408-445d-86dd-063aa13180e2/dcab90d0-6412-4eeb-8218-0c0b15cdd6ab"
-          (reference "C22") (unit 1)
-        )
-        (path "/271a56a4-fac2-444b-8acf-7cf36bf0ab17/997d7511-5408-445d-86dd-063aa13180e2/f2cea334-e45e-49d8-bc5b-499bf5169a47"
-          (reference "C25") (unit 1)
-        )
-      )
-    )
-  )
   (symbol (lib_id "Device:C") (at 165.1 71.12 0) (unit 1)
     (in_bom yes) (on_board yes) (dnp no) (fields_autoplaced)
@@
       (effects (font (size 1.27 1.27)) (justify left))
     )
-    (property "Value" "0,01uF 600V 1206 (GRM31BR72J103KW01L)" (at 168.91 72.39 0)
-      (effects (font (size 1.27 1.27)) (justify left))
-    )
-    (property "Footprint" "Capacitor_SMD:C_1206_3216Metric_Pad1.33x1.80mm_HandSolder" (at 166.0652 74.93 0)
+    (property "Value" "0,01uF 630V (CL11-103K/630V)" (at 168.91 72.39 0)
+      (effects (font (size 1.27 1.27)) (justify left))
+    )
+    (property "Footprint" "Capacitor_THT:C_Rect_L7.0mm_W4.5mm_P5.00mm" (at 166.0652 74.93 0)
       (effects (font (size 1.27 1.27)) hide)
     )
@@
     )
   )
+  (symbol (lib_id "Device:C") (at 119.38 80.01 0) (unit 1)
+    (in_bom yes) (on_board yes) (dnp no) (fields_autoplaced)
+    (property "Reference" "C19" (at 123.19 78.74 0)
+      (effects (font (size 1.27 1.27)) (justify left))
+    )
+    (property "Value" "0,01uF 630V (CL11-103K/630V)" (at 123.19 81.28 0)
+      (effects (font (size 1.27 1.27)) (justify left))
+    )
+    (property "Footprint" "Capacitor_THT:C_Rect_L7.0mm_W4.5mm_P5.00mm" (at 120.3452 83.82 0)
+      (effects (font (size 1.27 1.27)) hide)
+    )
+    (property "Datasheet" "~" (at 119.38 80.01 0)
+      (effects (font (size 1.27 1.27)) hide)
+    )
+    (pin "2")
+    (pin "1")
+    (instances
+      (project "triac_board"
+        (path "/271a56a4-fac2-444b-8acf-7cf36bf0ab17/997d7511-5408-445d-86dd-063aa13180e2/a92943f3-fb5f-4928-a4c6-18ad14104b9b"
+          (reference "C19") (unit 1)
+        )
+        (path "/271a56a4-fac2-444b-8acf-7cf36bf0ab17/997d7511-5408-445d-86dd-063aa13180e2/dcab90d0-6412-4eeb-8218-0c0b15cdd6ab"
+          (reference "C22") (unit 1)
+        )
+        (path "/271a56a4-fac2-444b-8acf-7cf36bf0ab17/997d7511-5408-445d-86dd-063aa13180e2/f2cea334-e45e-49d8-bc5b-499bf5169a47"
+          (reference "C25") (unit 1)
+        )
+        (path "/271a56a4-fac2-444b-8acf-7cf36bf0ab17/997d7511-5408-445d-86dd-063aa13180e2/63b095b4-3c9c-489d-b37a-8fc245f2b355"
+          (reference "C28") (unit 1)
+        )
+      )
+    )
+  )
   (symbol (lib_id "Device:C") (at 77.47 55.88 180) (unit 1)
     (in_bom yes) (on_board yes) (dnp no) (fields_autoplaced)
@@
       (effects (font (size 1.27 1.27)))
     )
-    (property "Value" "2512-1 кОм±5%-1 Вт" (at 125.73 48.26 90)
-      (effects (font (size 1.27 1.27)))
-    )
-    (property "Footprint" "Resistor_SMD:R_2512_6332Metric" (at 125.73 50.292 90)
+    (property "Value" "0207 MELF -1 кОм±5%-1 Вт" (at 125.73 48.26 90)
+      (effects (font (size 1.27 1.27)))
+    )
+    (property "Footprint" "Resistor_SMD:R_MELF_MMB-0207" (at 125.73 50.292 90)
       (effects (font (size 1.27 1.27)) hide)
     )
@@
       (effects (font (size 1.27 1.27)) (justify right))
     )
-    (property "Value" "2512-2 кОм±5%-1 Вт" (at 167.64 62.23 0)
+    (property "Value" "0207 MELF -2 кОм±5%-1 Вт" (at 167.64 62.23 0)
       (effects (font (size 1.27 1.27)) (justify right))
     )
-    (property "Footprint" "Resistor_SMD:R_2512_6332Metric" (at 166.878 60.96 90)
-      (effects (font (size 1.27 1.27)) hide)
-    )
+    (property "Footprint" "Resistor_SMD:R_MELF_MMB-0207" (at 166.878 60.96 90)
+      (effects (font (size 1.27 1.27)) hide)
+    )

Commit message: update schemas
Parts:
- renumbered C23 to C17, OC5 to OC2, Q1 to Q4
