File: Узел Питания и управления/Узел Питания и управления.kicad_sch (KiCad schematic)
At the start: 2 parts

Commit message: update schemas
Other:
- sheet Блоки питания AC|DC renamed Блоки питания AC\DC
- removed sheet QR_CODE LIGHT
- added sheet COFFEE_MACHINE (COFFE_MASHINE.kicad_sch)
- added sheet Схема стола (Table.kicad_sch)
- added sheet Таблица проводов 1 (ConnectionTable_1.kicad_sch)
- added sheet Таблица проводов 2 (ConnectionTable_2.kicad_sch)
- added sheet Таблица проводов 3 (ConnectionTable_3.kicad_sch)
- added sheet Таблица проводов 4 (ConnectionTable_4.kicad_sch)
- added sheet Таблица проводов 5 (ConnectionTable_5.kicad_sch)
- added sheet Таблица проводов 6 (ConnectionTable_6.kicad_sch)
- added sheet Таблица проводов 7 (ConnectionTable_7.kicad_sch)
- sheet Manipulator control ports: added Sync_IN, Sync_OUT; removed Manipulator_Control
- sheet MotherBord ports: added 9V_ANALOG, COFFEE_MACHINE_CTRL; removed 7V_ANALOG, COFFEE_MASHINE_CTRL
- sheet Router ports: added ROUTER_PS; removed 12V_IN
- sheet Server ports: added DMX; removed none
- sheet UPS ports: added 220V_MAN, 220V_SERVER; removed 220V_OUT
- sheet Блоки питания AC\DC ports: added 9V_ANALOG; removed 7V_ANALOG
- sheet Внешние подключения ports: added DMX_IN, HDMI_MONITOR_3, SINC_IN, SINC_OUT; removed 220_COFFEE_MASHINE, COFFEE_MASHINE_CTRL, Manipulator_Control, VGA_MONITOR_3
- sheet Освещение ports: added DMX_IN, DMX_OUT; removed RS485_IN
- sheet ЩИТ 220В ports: added 220V_LIGHT; removed GND
- moved on the sheet: 220_IN, Ethernet_OUT
