File: Узел нарезки/Connection table 2.kicad_sch (KiCad schematic)
At the start: 0 parts

Commit message: update schemas
Other:
- note added: "24AWG(0,2мм2)(белый)"
- note added: "24AWG(0,2мм2)(желтый)"
- note added: "24AWG(0,2мм2)(зеленый)"
- note added: "24AWG(0,2мм2)(красный)"
- note added: "24AWG(0,2мм2)(синий)"
- note added: "24AWG(0,2мм2)(черный)"
- note added: "AB_36V_J1/1"
- note added: "AB_36V_J1/2"
- note added: "AB_36V_J1/3"
- note added: "AB_36V_J1/4"
- note added: "AB_36V_J1/5"
- note added: "AB_36V_J1/6"
- note added: "AB_36V_J2/1"
- note added: "AB_36V_J2/2"
- note added: "AB_36V_J2/3"
- note added: "AB_36V_J2/4"
- note added: "AB_36V_J2/5"
- note added: "AB_36V_J2/6"
- note added: "DR_3_P3/1"
- note added: "DR_3_P3/2"
- note added: "DR_3_P3/3"
- note added: "DR_3_P4/1"
- note added: "DR_3_P4/2"
- note added: "DR_3_P4/3"
- note added: "DR_3_P4/4"
- note added: "DR_3_P4/5"
- note added: "DR_3_P4/6"
- note added: "PUMPS - разъем управления насосами соусов PUMP_(N) - насос номер N AB_36V - переходная колодка 36В DR_(N)_P(F) -драйвер номер N разъем драйвера F ST_(N) - плата управления драйвером шагового двигателя номер N"
- note added: "ST_3_J2/1"
- note added: "ST_3_J2/10"
- note added: "ST_3_J2/2"
- note added: "ST_3_J2/4"
- note added: "ST_3_J2/5"
- note added: "ST_3_J2/6"
- note added: "ST_3_J2/7"
- note added: "ST_3_J2/8"
- note added: "ST_3_J2/9"
- note added: "Объединить в один жгут"
- note added: "ПГВА 0,5 мм (красный)"
- note added: "ПГВА 0,5 мм (черный)"
- note added: "Установить гильзу НШВИ-0.34-8 с двух сторон и обжать"
- note added: "Установить гильзу НШВИ-0.5-8 с двух сторон и обжать"
- note removed: "0,2 мм"
- note removed: "0,35 мм"
- note removed: "0,5 мм"
- note removed: "16"
- note removed: "2,4"
- note removed: "31"
- note removed: "32"
- note removed: "74"
- note removed: "75"
- note removed: "76"
- note removed: "77"
- note removed: "78"
- note removed: "AB_50V_J1/1"
- note removed: "AB_50V_J1/2"
- note removed: "AB_50V_J1/3"
- note removed: "AB_50V_J1/4"
- note removed: "AB_50V_J1/5"
- note removed: "AB_50V_J1/6"
- note removed: "AB_50V_J2/1"
- note removed: "AB_50V_J2/2"
- note removed: "AB_50V_J2/3"
- note removed: "AB_50V_J2/4"
- note removed: "AB_50V_J2/5"
- note removed: "AB_50V_J2/6"
- note removed: "DC1_J3/1"
- note removed: "DC1_J3/2"
- note removed: "DC1_J4/1"
- note removed: "DC1_J4/2"
- note removed: "DC2_J3/1"
- note removed: "DC2_J3/2"
- note removed: "DC2_J4/1"
- note removed: "DC2_J4/2"
- note removed: "DC3_J3/1"
- note removed: "DC3_J3/2"
- note removed: "DC3_J4/1"
- note removed: "DC3_J4/2"
- note removed: "DC4_J3/1"
- note removed: "DC4_J3/2"
- note removed: "DC4_J4/1"
- note removed: "DC4_J4/2"
- note removed: "PUMPS - разъем управления насосами соусов PUMP_(N) - насос номер N AB_50V - переходная колодка 50В DR_(N)_P(F) -драйвер номер N разъем драйвера F ST_(N) - плата управления драйвером шагового двигателя номер N"
- note removed: "PUMPS/1"
- note removed: "PUMPS/10"
- note removed: "PUMPS/11"
- note removed: "PUMPS/12"
- note removed: "PUMPS/13"
- note removed: "PUMPS/14"
- note removed: "PUMPS/15"
- note removed: "PUMPS/16"
- note removed: "PUMPS/2"
- note removed: "PUMPS/3"
- note removed: "PUMPS/4"
- note removed: "PUMPS/5"
- note removed: "PUMPS/6"
- note removed: "PUMPS/7"
- note removed: "PUMPS/8"
- note removed: "PUMPS/9"
- note removed: "ПУТЬ"
