File: Узел нарезки/Connection table 4.kicad_sch (KiCad schematic)
At the start: 0 parts

Commit message: update schemas
Other:
- note added: "(Голубой)"
- note added: "(Зеленый)"
- note added: "(Красный)"
- note added: "(Черный)"
- note added: "**"
- note added: "** Провод идущий от датчика"
- note added: "*длину необходимо нарастить на расстоянии от двигателя: МОТ_3 - 50мм МОТ_4 - 150мм"
- note added: "105"
- note added: "106"
- note added: "107"
- note added: "108"
- note added: "109"
- note added: "110"
- note added: "1100*"
- note added: "111"
- note added: "112"
- note added: "113"
- note added: "114"
- note added: "115"
- note added: "116"
- note added: "117"
- note added: "118"
- note added: "800*"
- note added: "MOT_1 - Шаговый двигатель длинной оси ножа 23 MOT_2 - Шаговый двигатель длинной оси меандра nema23 MOT_3 - Шаговый двигатель короткой оси меандра nema 17 MOT_4 - Шаговый двигатель короткой оси ножа nema17 MOT_5 - Шаговый двигатель столика 1 nema14 MOT_6 - Шаговый двигатель столика 2 nema14"
- note added: "ПГВА 0,5 мм(Голубой)"
- note added: "ПГВА 0,5 мм(Зеленый)"
- note added: "ПГВА 0,5 мм(Красный)"
- note added: "ПГВА 0,5 мм(Черный)"
- note added: "Установить гильзу НШВИ-0.35-8"
- note added: "Установить гильзу НШВИ-0.5-8 со стороны драйвера"
- note removed: "0,2 мм"
- note removed: "0,5 мм"
- note removed: "1100"
- note removed: "145"
- note removed: "146"
- note removed: "147"
- note removed: "148"
- note removed: "149"
- note removed: "150"
- note removed: "151"
- note removed: "152"
- note removed: "153"
- note removed: "154"
- note removed: "155"
- note removed: "156"
- note removed: "157"
- note removed: "158"
- note removed: "800"
- note removed: "ПУТЬ"
