File: Узел печи/Table Connection2.kicad_sch (KiCad schematic)
At the start: 0 parts

Commit message: update schemas
Other:
- note added: "1500"
- note added: "79"
- note added: "80"
- note added: "81"
- note added: "ANALOG_J4/1"
- note added: "ANALOG_J4/2"
- note added: "ANALOG_J7/3"
- note added: "ANALOG_J8/1"
- note added: "ANALOG_J8/2"
- note added: "CurDET/2"
- note added: "L-FTP2-ST"
- note added: "T2_DATA(2)"
- note added: "T2_GND(1)"
- note added: "T2_VCC(3)"
- note added: "Витая пара (зеленый, белозеленый)"
- note added: "НВ-4-0.2 (Красный)"
- note added: "НВ-4-0.2 (красный)"
- note added: "НВ-4-0.2 (черный)"
- note added: "НВ-4-0.2 Желтый"
- note added: "НВ-4-0.2 Зеленый"
- note added: "НВ-4-0.2 Синий"
- note added: "НВ-4-0.2 Черный"
- note added: "Объединить в один жгут в термоусадку"
- note added: "ПВСнг(A)-LS 3x4 мм2"
- note added: "Со всех сторон гильза НШВИ-1.5-8"
- note added: "Установить НШВИ-0.34-8 с обоих сторон"
- note added: "Установить гильзу НШВИ-0.34-8"
- note added: "Установить гильзу НШВИ-0.34-8, со стороны реле наконечние М4"
- note added: "Установить гильзу НШВИ-1.5-8"
- note added: "Установить гильзы 4мм"
- note removed: "0,35 мм"
- note removed: "35"
- note removed: "350+внешнее"
- note removed: "36"
- note removed: "4 мм"
- note removed: "ANALOG_J11/1"
- note removed: "ANALOG_J11/2"
- note removed: "ANALOG_J9/1"
- note removed: "ANALOG_J9/2"
- note removed: "T2+"
- note removed: "T2-"
- note removed: "Витая пара"
- note removed: "Кабель для термопары"
- note removed: "ПУТЬ"
