File: Узел теста/Connection_Table1.kicad_sch (KiCad schematic)
At the start: 0 parts

Commit message: update schemas
Other:
- note added: "24AWG(0,2мм2)(белый)"
- note added: "24AWG(0,2мм2)(желтый)"
- note added: "24AWG(0,2мм2)(зеленый)"
- note added: "24AWG(0,2мм2)(красный)"
- note added: "24AWG(0,2мм2)(синий)"
- note added: "24AWG(0,2мм2)(черный)"
- note added: "Длина проводов не является окончательной и требует корректировки после первичной прокладки"
- note added: "Нумерация ячеек слева на право со стороны электроники"
- note added: "ПГВА 0,5 мм (красный)"
- note added: "ПГВА 0,5 мм (черный)"
- note added: "Установить гильзу НШВИ-0.34-8 с двух сторон и обжать"
- note added: "Установить гильзу НШВИ-0.5-12 с двух сторон и обжать"
- note removed: "0,2 мм"
- note removed: "0,35 мм"
- note removed: "0,75 мм"
- note removed: "ПУТЬ"
