File: Узел теста/Connection_Table3.kicad_sch (KiCad schematic)
At the start: 0 parts

Commit message: update schemas
Other:
- note added: "(Голубой)"
- note added: "(Зеленый)"
- note added: "(Красный)"
- note added: "(Черный)"
- note added: "**"
- note added: "** Провод идущий от датчика"
- note added: "*Наростить провода от двигателя до необходимой длины проводом ПГВА 0,5 мм"
- note added: "ПГВА 0,5 мм(Голубой)"
- note added: "ПГВА 0,5 мм(Зеленый)"
- note added: "ПГВА 0,5 мм(Красный)"
- note added: "ПГВА 0,5 мм(Черный)"
- note added: "Установить гильзу НШВИ-0.35-8"
- note added: "Установить гильзу НШВИ-0.5-8 со стороны разъёма драйвера"
- note removed: "0,2 мм"
- note removed: "0,5 мм"
- note removed: "ПУТЬ"
