File: Узел теста/MotherBord.kicad_sch (KiCad schematic)
At the start: 33 parts

Commit message: update schemas
Parts:
- renumbered DI_5_J11 to DI_1_J11, DI_2_J4 to DI_1_J4, DI_1_J11 to DI_2_J11, DI_3_J4 to DI_2_J4, DI_2_J11 to DI_3_J11, DI_4_J4 to DI_3_J4, DI_3_J11 to DI_4_J11, DI_5_J4 to DI_4_J4, DI_4_J11 to DI_5_J11, DI_1_J4 to DI_5_J4
Connections:
- net DI_1_IN+ renamed DI_1_J10+
- net DI_1_IN- renamed DI_1_J10-
- net DI_2_IN+ renamed DI_2_J10+
- net DI_2_IN- renamed DI_2_J10-
- net DI_3_IN+ renamed DI_3_J10+
- net DI_3_IN- renamed DI_3_J10-
- net DI_4_IN+ renamed DI_4_J10+
- net DI_4_IN- renamed DI_4_J10-
- net DI_5_IN+ renamed DI_5_J10+
- net DI_5_IN- renamed DI_5_J10-
- net LED_6_J1+ renamed LED_1_J1+
- net LED_6_J1- renamed LED_1_J1-
- net PHOTO_1_1 renamed PHOTO_6_1
- net PHOTO_1_2 renamed PHOTO_6_2
- net PHOTO_1_3 renamed PHOTO_6_3
- net PHOTO_1_4 renamed PHOTO_6_4
- net PHOTO_1_5 renamed PHOTO_6_5
- net PHOTO_1_6 renamed PHOTO_6_6
- net PHOTO_1_7 renamed PHOTO_6_7
- net PHOTO_1_8 renamed PHOTO_6_8
- net PHOTO_1_G renamed PHOTO_6_G
- net PHOTO_1_Vc renamed PHOTO_6_Vc
Other:
- moved on the sheet: DI_1_J11, DI_1_J4, DI_2_J11, DI_2_J4, DI_3_J11, DI_3_J4, DI_4_J11, DI_4_J4, DI_5_J11, DI_5_J4
