File: Узел упаковки/ConnectionTable2.kicad_sch (KiCad schematic)
At the start: 0 parts

Commit message: update schemas
Other:
- note added: "1000"
- note added: "1100"
- note added: "220V_OUT - разъем TE Connectivity 350780-1 Со стороны реле установить наконечник под М3"
- note added: "220V_OUT_L - 350780-1"
- note added: "220V_OUT_L/1"
- note added: "220V_OUT_L/2"
- note added: "220V_OUT_L/3"
- note added: "220V_OUT_L/4"
- note added: "220V_OUT_N - 350779-1"
- note added: "220V_OUT_N/1"
- note added: "220V_OUT_N/2"
- note added: "220V_OUT_N/3"
- note added: "220V_OUT_N/4"
- note added: "24AWG(0,2мм2)(белый)"
- note added: "24AWG(0,2мм2)(желтый)"
- note added: "24AWG(0,2мм2)(зеленый)"
- note added: "24AWG(0,2мм2)(красный)"
- note added: "24AWG(0,2мм2)(синий)"
- note added: "24AWG(0,2мм2)(черный)"
- note added: "3"
- note added: "36V_PACK - разъем GX12-3K"
- note added: "36V_PACK/1"
- note added: "36V_PACK/2"
- note added: "4"
- note added: "L-FTP2-ST"
- note added: "OUT_RS - разъем GX12-3A"
- note added: "OUT_RS/1"
- note added: "OUT_RS/2"
- note added: "Витая пара (зеленый, белозеленый)"
- note added: "НВ-4-0,35 (зеленый)"
- note added: "НВ-4-0,35 (красный)"
- note added: "НВ-4-0,35 (синий)"
- note added: "Объединить в один жгут"
- note added: "ПВС 2х0,5"
- note added: "Со стороны пайки"
- note added: "У платы DI установить гильзы НШВИ-0.35-8 Со стороны реле установить наконечник под М3"
- note added: "Установить гильзу НШВИ-0.34-8"
- note added: "Установить гильзу НШВИ-0.34-8 с двух сторон и обжать"
- note added: "Установить гильзу НШВИ-0.35-8 со стороны платы AB_220V 220V_OUT - разъем TE Connectivity 350779-1"
- note added: "Установить гильзу НШВИ-0.35-8 со стороны платы AB_220V Со стороны реле установить наконечник под М3"
- note added: "Установить гильзу НШВИ-0.5-8 со стороны драйвера"
- note added: "Установить кембрики со стороны разъема Объединить провода в термоусадку"
- note added: "ШВПМ 2 х 0,35(Красный)"
- note added: "ШВПМ 2 х 0,35(Черный)"
- note removed: "0,2 мм"
- note removed: "0,35 мм"
- note removed: "220V_OUT/1"
- note removed: "220V_OUT/2"
- note removed: "220V_OUT/3"
- note removed: "220V_OUT/4"
- note removed: "220V_OUT/5"
- note removed: "220V_OUT/6"
- note removed: "220V_OUT/7"
- note removed: "220V_OUT/8"
- note removed: "50V/1"
- note removed: "50V/2"
- note removed: "84"
- note removed: "85"
- note removed: "MOT_7_CONTR/3"
- note removed: "MOT_7_CONTR/4"
- note removed: "RS485/1"
- note removed: "RS485/2"
- note removed: "ST_1_J2/3"
- note removed: "Витая пара"
- note removed: "ПУТЬ"
