File: Узел упаковки/Connectors.kicad_sch (KiCad schematic)
At the start: 13 parts

Commit message: update schemas
Parts:
- removed 220V: ~, symbol Connector:Conn_01x02_(wide)
- removed 220V_OUT: ~, symbol Connector:Conn_01x08_(wide)
- removed DET_7_CAL, DET_7_MAX, DET_7_MIN: ~, symbol Connector:Conn_01x04_(wide)
- added 220V_IN, 220V_OUT_L, 220_OUT_N, QR_code1, QR_code2: ~, symbol Connector:Conn_01x04_(wide)
- added DET_7, SINC_IN, SINC_OUT: ~, symbol Connector:Conn_01x08_(wide)
- renumbered 24V_ANALOG1 to 24V_ANALOG_PACK, 50V_MOT_7 to 36V_MOT_7, 50V to 36V_PACK, RS485 to OUT_RS_PACK
Connections:
- net 220_IN_L: now also 220V_IN.1
- net 220_IN_N: now also 220V_IN.2
- net 220_OUT_1_L: now also 220V_OUT_L.1
- net 220_OUT_2_L: now also 220V_OUT_L.2
- net 220_OUT_3_L: now also 220V_OUT_L.3
- net 220_OUT_4_L: now also 220V_OUT_L.4
- net DET_7_MAX_BK: now also DET_7.6
- net DET_7_MAX_BL: now also DET_7.5
- net DET_7_MAX_BN: now also DET_7.8
- net DET_7_MAX_PK: now also DET_7.7
- net DET_7_MIN_BK: now also DET_7.2
- net DET_7_MIN_BL: now also DET_7.1
- net DET_7_MIN_BN: now also DET_7.4
- net DET_7_MIN_PK: now also DET_7.3
- net DR_1_50V+ renamed DR_1_36V+
- net DR_1_50V- renamed DR_1_36V-
- net MOT_7_50V+ renamed MOT_7_36V+
- net MOT_7_50V- renamed MOT_7_36V-
- new net 220_IN_G: 220V_IN.3
- new net 220_OUT_1_N: 220_OUT_N.1
- new net 220_OUT_2_N: 220_OUT_N.2
- new net 220_OUT_3_N: 220_OUT_N.3
- new net 220_OUT_4_N: 220_OUT_N.4
- new net QR_G_1: QR_code1.4
- new net QR_G_2: QR_code2.4
- new net QR_R_1: QR_code1.2
- new net QR_R_2: QR_code2.2
- new net QR_T_1: QR_code1.3
- new net QR_T_2: QR_code2.3
- new net QR_V_1: QR_code1.1
- new net QR_V_2: QR_code2.1
- new net SINC_IN_1+: SINC_IN.1
- new net SINC_IN_1-: SINC_IN.2
- new net SINC_IN_2+: SINC_IN.3
- new net SINC_IN_2-: SINC_IN.4
- new net SINC_IN_3+: SINC_IN.5
- new net SINC_IN_3-: SINC_IN.6
- new net SINC_O1+: SINC_OUT.1
- new net SINC_O1-: SINC_OUT.2
- new net SINC_O2+: SINC_OUT.3
- new net SINC_O2-: SINC_OUT.4
Other:
- moved on the sheet: 24V_ANALOG_PACK, 24V_DIG_PACK, 36V_PACK, OUT_RS_PACK
