File: Узел упаковки/Узел упаковки.kicad_sch (KiCad schematic)
At the start: 17 parts

Commit message: update schemas
Connections:
- net 220_IN_1_N renamed 220_OUT_1_N
- net 220_IN_2_N renamed 220_OUT_2_N
- net 220_IN_3_N renamed 220_OUT_3_N
- net 220_IN_4_N renamed 220_OUT_4_N
Other:
- added sheet ConnectionTable4 (ConnectionTable4.kicad_sch)
- sheet Внешние разъемы ports: added 36V, QR code, SINC; removed 50V
- sheet Материнская плата ports: added 36V, QR code, SINC; removed 50V
- moved on the sheet: AB_220V_J2+
